File: iroha60/pcb/iroha60.sch (KiCad schematic (older format))
At the start: 15 parts, among them J1 i2c-pin, J2 MJ-4PP-9, J3 i2c-pin, J4 LED, SW1 SW_PUSH, SW2 SW_PUSH, SW3 SW_PUSH, SW4 SW_PUSH, SW5 RESET_SW, U1 ProMicro

Commit message: wip
Parts:
- added D10, D11, D12, D13, D14, D15, D16, D17, D18, D19, D20, D21, D22, D23, D24, D25, D26, D27, D28, D29, D3, D30, D31, D32, D33, D34, D35, D36, D37, D38, D39, D4, D40, D41, D42, D43, D44, D45, D46, D47, D48, D49, D50, D51, D52, D53, D54, D55, D56, D57, D58, D59, D60, D61, D62, D7, D8, D9: D, symbol Device:D
- added J5: LED, symbol Connector_Generic:Conn_01x03
- added J6: MJ-4PP-9, symbol kbd:MJ-4PP-9
- added J7, J8: i2c-pin, symbol Connector_Generic:Conn_01x01
- added JP2: Jumper, symbol Device:Jumper
- added SW10, SW11, SW12, SW13, SW14, SW15, SW16, SW17, SW18, SW20, SW21, SW22, SW23, SW24, SW25, SW26, SW27, SW28, SW29, SW3, SW30, SW31, SW32, SW33, SW34, SW35, SW36, SW37, SW38, SW39, SW4, SW40, SW41, SW42, SW43, SW44, SW45, SW46, SW47, SW48, SW49, SW50, SW51, SW52, SW53, SW54, SW55, SW56, SW57, SW58, SW59, SW60, SW61, SW62, SW63, SW7, SW8, SW9: SW_PUSH, symbol kbd:SW_PUSH
- added SW64: RESET_SW, symbol kbd:SW_PUSH
- added U2: ProMicro, symbol kbd:ProMicro
- renumbered D3 to D2, D2 to D5, D4 to D6, J4 to J1, J1 to J3, J3 to J4, SW5 to SW19, SW3 to SW2, SW2 to SW5, SW4 to SW6
Connections:
- net GND: now also J5.1 (Pin_1), J6.C, SW64.2, U2.23 (GND), U2.3 (GND), U2.4 (GND)
- net VCC: now also J5.3 (Pin_3), J6.D, U2.21 (VCC)
- net col0: now also SW3.1, SW4.1
- net col1: now also SW7.1, SW8.1
- net row0: now also D14.1 (K), D19.1 (K), D24.1 (K), D9.1 (K)
- net row1: now also D10.1 (K), D15.1 (K), D20.1 (K), D25.1 (K)
- net row3: now reaches U1.10 (7/E6)
- net row3: now also D12.1 (K), D17.1 (K), D22.1 (K), D27.1 (K), D4.1 (K), D8.1 (K)
- net row4: now reaches U1.11 (8/B4)
- net row4: now also D13.1 (K), D18.1 (K), D23.1 (K), D28.1 (K)
- net col5: now reaches U1.15 (B3/14)
- net col5: now also SW25.1, SW26.1, SW27.1, SW28.1, SW29.1
- net col4: now reaches U1.16 (B1/15)
- net col4: now also SW20.1, SW21.1, SW22.1, SW23.1, SW24.1
- net col3: now reaches U1.17 (F7/A0)
- net col3: now also SW14.1, SW15.1, SW16.1, SW17.1, SW18.1
- net col2: now reaches U1.18 (F6/A1)
- net col2: now also SW10.1, SW11.1, SW12.1, SW13.1, SW9.1
- net row2: now reaches U1.9 (6/D7)
- net row2: now also D11.1 (K), D16.1 (K), D21.1 (K), D26.1 (K), D3.1 (K), D7.1 (K)
- new net: D9.2 (A), SW9.2
- new net: D14.2 (A), SW14.2
- new net: D19.2 (A), SW20.2
- new net: D24.2 (A), SW25.2
- new net: D10.2 (A), SW10.2
- new net: D15.2 (A), SW15.2
- new net: D20.2 (A), SW21.2
- new net: D25.2 (A), SW26.2
- new net: D3.2 (A), SW3.2
- new net: D7.2 (A), SW7.2
- new net: D11.2 (A), SW11.2
- new net: D16.2 (A), SW16.2
- new net: D21.2 (A), SW22.2
- new net: D26.2 (A), SW27.2
- new net: D4.2 (A), SW4.2
- new net: D8.2 (A), SW8.2
- new net: D12.2 (A), SW12.2
- new net: D17.2 (A), SW17.2
- new net: D22.2 (A), SW23.2
- new net: D27.2 (A), SW28.2
- new net: D28.2 (A), SW29.2
- new net: D23.2 (A), SW24.2
- new net: D18.2 (A), SW18.2
- new net: D13.2 (A), SW13.2
- new net: D29.2 (A), SW30.2
- new net: D30.2 (A), SW31.2
- new net: D32.2 (A), SW33.2
- new net: D37.2 (A), SW38.2
- new net: D42.2 (A), SW43.2
- new net: D47.2 (A), SW48.2
- new net: D51.2 (A), SW52.2
- new net: D55.2 (A), SW56.2
- new net: D59.2 (A), SW60.2
- new net: D31.2 (A), SW32.2
- new net: D33.2 (A), SW34.2
- new net: D38.2 (A), SW39.2
- new net: D43.2 (A), SW44.2
- new net: D48.2 (A), SW49.2
- new net: D52.2 (A), SW53.2
- new net: D56.2 (A), SW57.2
- new net: D60.2 (A), SW61.2
- new net: D34.2 (A), SW35.2
- new net: D39.2 (A), SW40.2
- new net: D44.2 (A), SW45.2
- new net: D49.2 (A), SW50.2
- new net: D53.2 (A), SW54.2
- new net: D57.2 (A), SW58.2
- new net: D61.2 (A), SW62.2
- new net: D35.2 (A), SW36.2
- new net: D40.2 (A), SW41.2
- new net: D45.2 (A), SW46.2
- new net: D50.2 (A), SW51.2
- new net: D54.2 (A), SW55.2
- new net: D58.2 (A), SW59.2
- new net: D62.2 (A), SW63.2
- new net: D36.2 (A), SW37.2
- new net: D41.2 (A), SW42.2
- new net: D46.2 (A), SW47.2
- new net: J6.A, J7.1 (Pin_1)
- new net: J6.B, J8.1 (Pin_1), JP2.2
- new net R-col0: SW30.1, U2.20 (F4/A3)
- new net R-col1: SW31.1, SW32.1, U2.19 (F5/A2)
- new net R-col2: SW33.1, SW34.1, SW35.1, SW36.1, SW37.1, U2.18 (F6/A1)
- new net R-col3: SW38.1, SW39.1, SW40.1, SW41.1, SW42.1, U2.17 (F7/A0)
- new net R-col4: SW43.1, SW44.1, SW45.1, SW46.1, SW47.1, U2.16 (B1/15)
- new net R-col5: SW48.1, SW49.1, SW50.1, SW51.1, U2.15 (B3/14)
- new net R-col6: SW52.1, SW53.1, SW54.1, SW55.1, U2.14 (B2/16)
- new net R-col7: SW56.1, SW57.1, SW58.1, SW59.1, U2.13 (B6/10)
- new net R-col8: SW60.1, SW61.1, SW62.1, SW63.1, U2.12 (9/B5)
- new net R-data: JP2.1, U2.2 (RX1/D2)
- new net R-led: J5.2 (Pin_2), U2.1 (TX0/D3)
- new net R-reset: SW64.1, U2.22 (RST)
- new net R-row0: D29.1 (K), D30.1 (K), D32.1 (K), D37.1 (K), D42.1 (K), D47.1 (K), D51.1 (K), D55.1 (K), D59.1 (K), U2.7 (4/D4)
- new net R-row1: D31.1 (K), D33.1 (K), D38.1 (K), D43.1 (K), D48.1 (K), D52.1 (K), D56.1 (K), D60.1 (K), U2.8 (5/C6)
- new net R-row2: D34.1 (K), D39.1 (K), D44.1 (K), D49.1 (K), D53.1 (K), D57.1 (K), D61.1 (K), U2.9 (6/D7)
- new net R-row3: D35.1 (K), D40.1 (K), D45.1 (K), D50.1 (K), D54.1 (K), D58.1 (K), D62.1 (K), U2.10 (7/E6)
- new net R-row4: D36.1 (K), D41.1 (K), D46.1 (K), U2.11 (8/B4)
- no-connect marks 13 -> 9
Other:
- moved on the sheet: D1, D2, D5, D6, J1, J2, J3, J4, JP1, SW1, SW19, SW2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

Commit message: wip
Parts:
- added JP3: Jumper, kbd:Jumper, symbol Device:Jumper
- D1, D10, D11, D12, D13, D14, D15, D16, D17, D18, D19, D2, D20, D21, D22, D23, D24, D25, D26, D27, D28, D29, D3, D30, D31, D32, D33, D34, D35, D36, D37, D38, D39, D4, D40, D41, D42, D43, D44, D45, D46, D47, D48, D49, D5, D50, D51, D52, D53, D54, D55, D56, D57, D58, D59, D6, D60, D61, D62, D7, D8, D9: footprint (none) -> kbd:D3_TH_SMD
- J1, J5: footprint (none) -> kbd:StripLED_1side
- J2, J6: footprint (none) -> kbd:MJ-4PP-9_1side
- J3, J4, J7, J8: footprint (none) -> kbd:1pin_conn
- JP1, JP2: footprint (none) -> kbd:Jumper
- SW1, SW10, SW11, SW12, SW13, SW14, SW15, SW16, SW17, SW18, SW2, SW20, SW21, SW22, SW23, SW24, SW25, SW26, SW27, SW28, SW29, SW3, SW30, SW31, SW32, SW33, SW34, SW35, SW36, SW37, SW38, SW39, SW4, SW40, SW41, SW42, SW43, SW44, SW45, SW46, SW47, SW48, SW49, SW5, SW50, SW51, SW52, SW53, SW54, SW55, SW56, SW57, SW58, SW59, SW6, SW60, SW61, SW62, SW63, SW7, SW8, SW9: footprint (none) -> Keebio-Parts:MX-Alps-Choc-1U-NoLED
- SW19, SW64: footprint (none) -> kbd:ResetSW_1side
- U1, U2: footprint (none) -> kbd:ProMicro_v3
Connections:
- net R-data: now also JP3.1
- net col0 renamed L-col0
- net col1 renamed L-col1
- net col2 renamed L-col2
- net col3 renamed L-col3
- net col4 renamed L-col4
- net col5 renamed L-col5
- net data renamed L-data
- net L-data: now also JP3.2
- net led renamed L-led
- net row0 renamed L-row0
- net row1 renamed L-row1
- net row2 renamed L-row2
- net row3 renamed L-row3
- net row4 renamed L-row4

Commit message: wip
Parts:
- removed D13: D, kbd:D3_TH_SMD, symbol Device:D
- removed SW13: SW_PUSH, Keebio-Parts:MX-Alps-Choc-1U-NoLED, symbol kbd:SW_PUSH
- added D38, D47, D55, D63, D67, D68, D69, D7: D, kbd:D3_TH_SMD, symbol Device:D
- added SW38, SW47, SW55, SW63, SW67, SW68, SW69, SW7: SW_PUSH, MX_Alps_Hybrid:MX-1U-NoLED, symbol kbd:SW_PUSH
- SW1, SW10: footprint Keebio-Parts:MX-Alps-Choc-1U-NoLED -> MX_Alps_Hybrid:MX-1U-NoLED
- SW11: renamed from SW15; footprint Keebio-Parts:MX-Alps-Choc-1U-NoLED -> MX_Alps_Hybrid:MX-1U-NoLED
- SW12: renamed from SW21; footprint Keebio-Parts:MX-Alps-Choc-1U-NoLED -> MX_Alps_Hybrid:MX-1U-NoLED
- SW13: renamed from SW26; footprint Keebio-Parts:MX-Alps-Choc-1U-NoLED -> MX_Alps_Hybrid:MX-1U-NoLED
- SW14: renamed from SW3; footprint Keebio-Parts:MX-Alps-Choc-1U-NoLED -> MX_Alps_Hybrid:MX-1.75U-NoLED
- SW15: renamed from SW7; footprint Keebio-Parts:MX-Alps-Choc-1U-NoLED -> MX_Alps_Hybrid:MX-1U-NoLED
- SW16: renamed from SW11; footprint Keebio-Parts:MX-Alps-Choc-1U-NoLED -> MX_Alps_Hybrid:MX-1U-NoLED
- SW17: renamed from SW16; footprint Keebio-Parts:MX-Alps-Choc-1U-NoLED -> MX_Alps_Hybrid:MX-1U-NoLED
- SW18: renamed from SW22; footprint Keebio-Parts:MX-Alps-Choc-1U-NoLED -> MX_Alps_Hybrid:MX-1U-NoLED
- SW19: renamed from SW27; footprint Keebio-Parts:MX-Alps-Choc-1U-NoLED -> MX_Alps_Hybrid:MX-1U-NoLED
- SW2: renamed from SW5; footprint Keebio-Parts:MX-Alps-Choc-1U-NoLED -> MX_Alps_Hybrid:MX-1U-NoLED
- SW20: renamed from SW4; footprint Keebio-Parts:MX-Alps-Choc-1U-NoLED -> MX_Alps_Hybrid:MX-2.25U-NoLED
- SW21: renamed from SW8; footprint Keebio-Parts:MX-Alps-Choc-1U-NoLED -> MX_Alps_Hybrid:MX-1U-NoLED
- SW22: renamed from SW12; footprint Keebio-Parts:MX-Alps-Choc-1U-NoLED -> MX_Alps_Hybrid:MX-1U-NoLED
- SW23: renamed from SW17; footprint Keebio-Parts:MX-Alps-Choc-1U-NoLED -> MX_Alps_Hybrid:MX-1U-NoLED
- SW24: renamed from SW23; footprint Keebio-Parts:MX-Alps-Choc-1U-NoLED -> MX_Alps_Hybrid:MX-1U-NoLED
- SW25: renamed from SW28; footprint Keebio-Parts:MX-Alps-Choc-1U-NoLED -> MX_Alps_Hybrid:MX-1U-NoLED
- SW26: renamed from SW18; footprint Keebio-Parts:MX-Alps-Choc-1U-NoLED -> MX_Alps_Hybrid:MX-1U-NoLED
- SW27: renamed from SW24; footprint Keebio-Parts:MX-Alps-Choc-1U-NoLED -> MX_Alps_Hybrid:MX-1.5U-NoLED
- SW28: renamed from SW29; footprint Keebio-Parts:MX-Alps-Choc-1U-NoLED -> MX_Alps_Hybrid:MX-2.75U-NoLED
- SW29: renamed from SW30; footprint Keebio-Parts:MX-Alps-Choc-1U-NoLED -> MX_Alps_Hybrid:MX-1U-NoLED
- SW3: renamed from SW9; footprint Keebio-Parts:MX-Alps-Choc-1U-NoLED -> MX_Alps_Hybrid:MX-1U-NoLED
- SW30: renamed from SW31; footprint Keebio-Parts:MX-Alps-Choc-1U-NoLED -> MX_Alps_Hybrid:MX-1U-NoLED
- SW31: renamed from SW33; footprint Keebio-Parts:MX-Alps-Choc-1U-NoLED -> MX_Alps_Hybrid:MX-1U-NoLED
- SW32: renamed from SW38; footprint Keebio-Parts:MX-Alps-Choc-1U-NoLED -> MX_Alps_Hybrid:MX-1U-NoLED
- SW33: renamed from SW43; footprint Keebio-Parts:MX-Alps-Choc-1U-NoLED -> MX_Alps_Hybrid:MX-1U-NoLED
- SW34: renamed from SW48; footprint Keebio-Parts:MX-Alps-Choc-1U-NoLED -> MX_Alps_Hybrid:MX-1U-NoLED
- SW35: renamed from SW52; footprint Keebio-Parts:MX-Alps-Choc-1U-NoLED -> MX_Alps_Hybrid:MX-1U-NoLED
- SW36: renamed from SW56; footprint Keebio-Parts:MX-Alps-Choc-1U-NoLED -> MX_Alps_Hybrid:MX-1U-NoLED
- SW37: renamed from SW60; footprint Keebio-Parts:MX-Alps-Choc-1U-NoLED -> MX_Alps_Hybrid:MX-1U-NoLED
- SW39: renamed from SW32; footprint Keebio-Parts:MX-Alps-Choc-1U-NoLED -> MX_Alps_Hybrid:MX-1U-NoLED
- SW4: renamed from SW14; footprint Keebio-Parts:MX-Alps-Choc-1U-NoLED -> MX_Alps_Hybrid:MX-1U-NoLED
- SW40: renamed from SW34; footprint Keebio-Parts:MX-Alps-Choc-1U-NoLED -> MX_Alps_Hybrid:MX-1U-NoLED
- SW41: renamed from SW39; footprint Keebio-Parts:MX-Alps-Choc-1U-NoLED -> MX_Alps_Hybrid:MX-1U-NoLED
- SW42: renamed from SW44; footprint Keebio-Parts:MX-Alps-Choc-1U-NoLED -> MX_Alps_Hybrid:MX-1U-NoLED
- SW43: renamed from SW49; footprint Keebio-Parts:MX-Alps-Choc-1U-NoLED -> MX_Alps_Hybrid:MX-1U-NoLED
- SW44: renamed from SW53; footprint Keebio-Parts:MX-Alps-Choc-1U-NoLED -> MX_Alps_Hybrid:MX-1U-NoLED
- SW45: renamed from SW57; footprint Keebio-Parts:MX-Alps-Choc-1U-NoLED -> MX_Alps_Hybrid:MX-1.5U-NoLED
- SW46: renamed from SW61; footprint Keebio-Parts:MX-Alps-Choc-1U-NoLED -> MX_Alps_Hybrid:MX-1U-NoLED
- SW48: renamed from SW35; footprint Keebio-Parts:MX-Alps-Choc-1U-NoLED -> MX_Alps_Hybrid:MX-1U-NoLED
- SW49: renamed from SW40; footprint Keebio-Parts:MX-Alps-Choc-1U-NoLED -> MX_Alps_Hybrid:MX-1U-NoLED
- SW5: renamed from SW20; footprint Keebio-Parts:MX-Alps-Choc-1U-NoLED -> MX_Alps_Hybrid:MX-1U-NoLED
- SW50: renamed from SW45; footprint Keebio-Parts:MX-Alps-Choc-1U-NoLED -> MX_Alps_Hybrid:MX-1U-NoLED
- SW51: renamed from SW50; footprint Keebio-Parts:MX-Alps-Choc-1U-NoLED -> MX_Alps_Hybrid:MX-1U-NoLED
- SW52: renamed from SW54; footprint Keebio-Parts:MX-Alps-Choc-1U-NoLED -> MX_Alps_Hybrid:MX-1U-NoLED
- SW53: renamed from SW58; footprint Keebio-Parts:MX-Alps-Choc-1U-NoLED -> MX_Alps_Hybrid:MX-2.25U-NoLED
- SW54: renamed from SW62; footprint Keebio-Parts:MX-Alps-Choc-1U-NoLED -> MX_Alps_Hybrid:MX-1U-NoLED
- SW56: renamed from SW36; footprint Keebio-Parts:MX-Alps-Choc-1U-NoLED -> MX_Alps_Hybrid:MX-1U-NoLED
- SW57: renamed from SW41; footprint Keebio-Parts:MX-Alps-Choc-1U-NoLED -> MX_Alps_Hybrid:MX-1U-NoLED
- SW58: renamed from SW46; footprint Keebio-Parts:MX-Alps-Choc-1U-NoLED -> MX_Alps_Hybrid:MX-1U-NoLED
- SW59: renamed from SW51; footprint Keebio-Parts:MX-Alps-Choc-1U-NoLED -> MX_Alps_Hybrid:MX-1U-NoLED
- SW6: renamed from SW25; footprint Keebio-Parts:MX-Alps-Choc-1U-NoLED -> MX_Alps_Hybrid:MX-1U-NoLED
- SW60: renamed from SW55; footprint Keebio-Parts:MX-Alps-Choc-1U-NoLED -> MX_Alps_Hybrid:MX-1.75U-NoLED
- SW61: renamed from SW59; footprint Keebio-Parts:MX-Alps-Choc-1U-NoLED -> MX_Alps_Hybrid:MX-1U-NoLED
- SW62: renamed from SW63; footprint Keebio-Parts:MX-Alps-Choc-1U-NoLED -> MX_Alps_Hybrid:MX-1U-NoLED
- SW64: renamed from SW37; footprint Keebio-Parts:MX-Alps-Choc-1U-NoLED -> MX_Alps_Hybrid:MX-2.25U-NoLED
- SW65: renamed from SW42; footprint Keebio-Parts:MX-Alps-Choc-1U-NoLED -> MX_Alps_Hybrid:MX-1.5U-NoLED
- SW66: renamed from SW47; footprint Keebio-Parts:MX-Alps-Choc-1U-NoLED -> MX_Alps_Hybrid:MX-1U-NoLED
- SW8: renamed from SW2; footprint Keebio-Parts:MX-Alps-Choc-1U-NoLED -> MX_Alps_Hybrid:MX-1.5U-NoLED
- SW9: renamed from SW6; footprint Keebio-Parts:MX-Alps-Choc-1U-NoLED -> MX_Alps_Hybrid:MX-1U-NoLED
- renumbered D15 to D11, D20 to D12, D25 to D13, D3 to D14, D7 to D15, D11 to D16, D16 to D17, D21 to D18, D26 to D19, D5 to D2, D4 to D20, D8 to D21, D12 to D22, D17 to D23, D22 to D24, D27 to D25, D18 to D26, D23 to D27, D9 to D3, D32 to D31, D37 to D32, D42 to D33, D47 to D34, D51 to D35, D55 to D36, D59 to D37, D31 to D39, D14 to D4, D33 to D40, D38 to D41, D43 to D42, D48 to D43, D52 to D44, D56 to D45, D60 to D46, D34 to D48, D39 to D49, D19 to D5, D44 to D50, D49 to D51, D53 to D52, D57 to D53, D61 to D54, D35 to D56, D40 to D57, D45 to D58, D50 to D59, D24 to D6, D54 to D60, D58 to D61, D36 to D64, D41 to D65, D46 to D66, D2 to D8, D6 to D9, J3 to J1, J4 to J3, J1 to J4, J7 to J5, J8 to J7, J5 to J8, SW19 to SW70, SW64 to SW71
Connections:
- net L-col0: no longer SW14.1, SW20.1, SW8.1
- net L-col1: now also SW14.1, SW20.1, SW8.1; no longer SW15.1, SW21.1, SW9.1
- net L-col2: now also SW15.1, SW21.1, SW9.1; no longer SW10.1, SW16.1, SW22.1
- net L-col3: now also SW10.1, SW16.1, SW22.1; no longer SW11.1, SW17.1, SW23.1, SW26.1
- net L-col4: now also SW11.1, SW17.1, SW23.1, SW26.1; no longer SW12.1, SW18.1, SW24.1, SW27.1
- net L-col5: now also SW12.1, SW18.1, SW24.1, SW27.1; no longer SW13.1, SW19.1, SW25.1, SW28.1
- net L-row0: now also D7.1 (K)
- net R-col0: now also SW38.1
- net R-col1: now also SW47.1, SW55.1, SW63.1
- net R-col6: now also SW67.1
- net R-col7: now also SW68.1
- net R-col8: now also SW69.1
- net R-row1: now also D38.1 (K)
- net R-row2: now also D47.1 (K)
- net R-row3: now also D55.1 (K)
- net R-row4: now also D63.1 (K), D67.1 (K), D68.1 (K), D69.1 (K)
- net L-col6: now reaches U1.14 (B2/16)
- net L-col6: now also SW13.1, SW19.1, SW25.1, SW28.1, SW7.1
- new net: D7.2 (A), SW7.2
- new net: D38.2 (A), SW38.2
- new net: D47.2 (A), SW47.2
- new net: D55.2 (A), SW55.2
- new net: D69.2 (A), SW69.2
- new net: D68.2 (A), SW68.2
- new net: D67.2 (A), SW67.2
- new net: D63.2 (A), SW63.2
- no-connect marks 9 -> 8
Other:
- moved on the sheet: D1, D10, D11, D12, D13, D14, D15, D16, D17, D18, D19, D2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
