File: iroha60/pcb/iroha60.kicad_pcb (KiCad board)
At the start: 2 copper layers, 139 parts, among them J1 LED, J2 MJ-4PP-9, J3 i2c-pin, J4 i2c-pin, J5 LED, J6 MJ-4PP-9, J7 i2c-pin, J8 i2c-pin, SW1 SW_PUSH, SW10 SW_PUSH, SW11 SW_PUSH, SW12 SW_PUSH, SW13 SW_PUSH, SW14 SW_PUSH, SW15 SW_PUSH, SW16 SW_PUSH, SW17 SW_PUSH, SW18 SW_PUSH, SW19 RESET_SW, SW2 SW_PUSH, SW20 SW_PUSH, SW21 SW_PUSH, SW22 SW_PUSH, SW23 SW_PUSH, SW24 SW_PUSH, SW25 SW_PUSH, SW26 SW_PUSH, SW27 SW_PUSH, SW28 SW_PUSH, SW29 SW_PUSH, SW3 SW_PUSH, SW30 SW_PUSH, SW31 SW_PUSH, SW32 SW_PUSH, SW33 SW_PUSH, SW34 SW_PUSH, SW35 SW_PUSH, SW36 SW_PUSH, SW37 SW_PUSH, SW38 SW_PUSH, SW39 SW_PUSH, SW4 SW_PUSH, SW40 SW_PUSH, SW41 SW_PUSH, SW42 SW_PUSH, SW43 SW_PUSH, SW44 SW_PUSH, SW45 SW_PUSH, SW46 SW_PUSH, SW47 SW_PUSH, SW48 SW_PUSH, SW49 SW_PUSH, SW5 SW_PUSH, SW50 SW_PUSH, SW51 SW_PUSH, SW52 SW_PUSH, SW53 SW_PUSH, SW54 SW_PUSH, SW55 SW_PUSH, SW56 SW_PUSH, SW57 SW_PUSH, SW58 SW_PUSH, SW59 SW_PUSH, SW6 SW_PUSH, SW60 SW_PUSH, SW61 SW_PUSH, SW62 SW_PUSH, SW63 SW_PUSH, SW64 RESET_SW, SW7 SW_PUSH, SW8 SW_PUSH, SW9 SW_PUSH, U1 ProMicro, U2 ProMicro

Commit message: wip
Parts:
- added D63: D, kbd:D3_TH_SMD, F.Cu at (166.9, 106.1)
- added D64: D, kbd:D3_TH_SMD, F.Cu at (171.9, 106.1)
- added D65: D, kbd:D3_TH_SMD, F.Cu at (217.2, 106.1)
- added D66: D, kbd:D3_TH_SMD, F.Cu at (241.0, 106.1)
- added D67: D, kbd:D3_TH_SMD, F.Cu at (269.6, 106.1)
- added D68: D, kbd:D3_TH_SMD, F.Cu at (288.6, 106.1)
- added D69: D, kbd:D3_TH_SMD, F.Cu at (307.7, 106.1)
- added SW65: SW_PUSH, MX_Alps_Hybrid:MX-1.5U-NoLED, F.Cu at (225.4, 106.1)
- added SW66: SW_PUSH, MX_Alps_Hybrid:MX-1U-NoLED, F.Cu at (249.2, 106.1)
- added SW67: SW_PUSH, MX_Alps_Hybrid:MX-1U-NoLED, F.Cu at (277.8, 106.1)
- added SW68: SW_PUSH, MX_Alps_Hybrid:MX-1U-NoLED, F.Cu at (296.8, 106.1)
- added SW69: SW_PUSH, MX_Alps_Hybrid:MX-1U-NoLED, F.Cu at (315.9, 106.1)
- added SW70: RESET_SW, kbd:ResetSW_1side, B.Cu at (22.3, 58.5)
- added SW71: RESET_SW, kbd:ResetSW_1side, B.Cu at (323.7, 58.5)
- J1, J5: value LED -> i2c-pin; footprint kbd:StripLED_1side -> kbd:1pin_conn
- J2, J6, U1, U2: moved to B.Cu
- J4, J8: value i2c-pin -> LED; footprint kbd:1pin_conn -> kbd:StripLED_1side; moved to B.Cu
- SW1, SW10, SW11, SW12, SW13, SW15, SW16, SW17, SW18, SW2, SW21, SW22, SW23, SW24, SW25, SW26, SW29, SW3, SW30, SW31, SW32, SW33, SW34, SW35, SW36, SW37, SW38, SW39, SW4, SW40, SW41, SW42, SW43, SW44, SW46, SW47, SW48, SW49, SW5, SW50, SW51, SW52, SW54, SW55, SW56, SW57, SW58, SW59, SW6, SW61, SW62, SW63, SW7, SW9: footprint Keebio-Parts:MX-Alps-Choc-1U-NoLED -> MX_Alps_Hybrid:MX-1U-NoLED
- SW14, SW60: footprint Keebio-Parts:MX-Alps-Choc-1U-NoLED -> MX_Alps_Hybrid:MX-1.75U-NoLED
- SW19: value RESET_SW -> SW_PUSH; footprint kbd:ResetSW_1side -> MX_Alps_Hybrid:MX-1U-NoLED
- SW20: footprint Keebio-Parts:MX-Alps-Choc-1U-NoLED -> MX_Alps_Hybrid:MX-2.25U-ReversedStabilizers-NoLED
- SW27, SW45, SW8: footprint Keebio-Parts:MX-Alps-Choc-1U-NoLED -> MX_Alps_Hybrid:MX-1.5U-NoLED
- SW28: footprint Keebio-Parts:MX-Alps-Choc-1U-NoLED -> MX_Alps_Hybrid:MX-2.75U-ReversedStabilizers-NoLED
- SW53: footprint Keebio-Parts:MX-Alps-Choc-1U-NoLED -> MX_Alps_Hybrid:MX-2.25U-NoLED
- SW64: value RESET_SW -> SW_PUSH; footprint kbd:ResetSW_1side -> MX_Alps_Hybrid:MX-2.25U-ReversedStabilizers-NoLED
- moved D35 299.0 mm to (269.6, 29.9), turned to 90 degrees
- moved SW62 294.6 mm to (315.9, 87.1)
- moved D54 293.2 mm to (307.7, 68.0), turned to 90 degrees
- moved SW46 291.2 mm to (315.9, 49.0)
- moved U2 284.1 mm to (305.8, 29.8), turned to 90 degrees
- moved D46 270.9 mm to (307.7, 49.0), turned to 90 degrees
- moved D62 270.8 mm to (324.3, 87.1), turned to 90 degrees
- moved SW44 259.5 mm to (268.2, 49.0)
- moved D45 258.0 mm to (279.1, 49.0), turned to 90 degrees
- moved SW45 252.0 mm to (292.1, 49.0)
- moved D53 251.4 mm to (267.2, 68.0), turned to 90 degrees
- moved D61 249.3 mm to (288.6, 87.1), turned to 90 degrees
- moved JP1 247.5 mm to (22.2, 43.9), turned to 270 degrees
- moved J3 247.5 mm to (22.2, 46.6), turned to 90 degrees
- moved D36 246.3 mm to (300.5, 49.0), turned to 90 degrees
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Connections:
- D11 pad 1: L-row2 -> L-row1
- D12 pad 1: L-row3 -> L-row1
- D13 pad 1: L-row4 -> L-row1
- D14 pad 1: L-row0 -> L-row2
- D15 pad 1: L-row1 -> L-row2
- D17 pad 1: L-row3 -> L-row2
- D18 pad 1: L-row4 -> L-row2
- D19 pad 1: L-row0 -> L-row2
- D2 pad 1: L-row1 -> L-row0
- D20 pad 1: L-row1 -> L-row3
- D21 pad 1: L-row2 -> L-row3
- D23 pad 1: L-row4 -> L-row3
- D24 pad 1: L-row0 -> L-row3
- D25 pad 1: L-row1 -> L-row3
- D26 pad 1: L-row2 -> L-row4
- D27 pad 1: L-row3 -> L-row4
- D3 pad 1: L-row2 -> L-row0
- D31 pad 1: R-row1 -> R-row0
- D33 pad 1: R-row1 -> R-row0
- D34 pad 1: R-row2 -> R-row0
- D35 pad 1: R-row3 -> R-row0
- D36 pad 1: R-row4 -> R-row0
- D39 pad 1: R-row2 -> R-row1
- D4 pad 1: L-row3 -> L-row0
- D40 pad 1: R-row3 -> R-row1
- D41 pad 1: R-row4 -> R-row1
- D42 pad 1: R-row0 -> R-row1
- D44 pad 1: R-row2 -> R-row1
- D45 pad 1: R-row3 -> R-row1
- D46 pad 1: R-row4 -> R-row1
- D47 pad 1: R-row0 -> R-row2
- D48 pad 1: R-row1 -> R-row2
- D50 pad 1: R-row3 -> R-row2
- D51 pad 1: R-row0 -> R-row2
- D52 pad 1: R-row1 -> R-row2
- D54 pad 1: R-row3 -> R-row2
- D55 pad 1: R-row0 -> R-row3
- D56 pad 1: R-row1 -> R-row3
- D57 pad 1: R-row2 -> R-row3
- D59 pad 1: R-row0 -> R-row3
- D6 pad 1: L-row1 -> L-row0
- D60 pad 1: R-row1 -> R-row3
- D61 pad 1: R-row2 -> R-row3
- D7 pad 1: L-row2 -> L-row0
- D8 pad 1: L-row3 -> L-row1
- D9 pad 1: L-row0 -> L-row1
- J1 pad 1: GND -> Net-(J1-Pad1)
- J2 pad A: Net-(J2-PadA) -> Net-(J1-Pad1)
- J3 pad 1: Net-(J2-PadA) -> Net-(J2-PadB)
- J4 pad 1: Net-(J2-PadB) -> GND
- J5 pad 1: GND -> Net-(J5-Pad1)
- J6 pad A: Net-(J6-PadA) -> Net-(J5-Pad1)
- J7 pad 1: Net-(J6-PadA) -> Net-(J6-PadB)
- J8 pad 1: Net-(J6-PadB) -> GND
- SW10 pad 1: L-col2 -> L-col3
- SW11 pad 1: L-col2 -> L-col4
- SW12 pad 1: L-col2 -> L-col5
- SW13 pad 1: L-col2 -> L-col6
- SW14 pad 1: L-col3 -> L-col1
- SW15 pad 1: L-col3 -> L-col2
- SW17 pad 1: L-col3 -> L-col4
- SW18 pad 1: L-col3 -> L-col5
- SW19 pad 1: reset -> L-col6
- SW19 pad 2: GND -> Net-(D19-Pad2)
- SW2 pad 1: L-col0 -> L-col1
- SW20 pad 1: L-col4 -> L-col1
- SW20 pad 2: Net-(D19-Pad2) -> Net-(D20-Pad2)
- SW21 pad 1: L-col4 -> L-col2
- SW21 pad 2: Net-(D20-Pad2) -> Net-(D21-Pad2)
- SW22 pad 1: L-col4 -> L-col3
- SW22 pad 2: Net-(D21-Pad2) -> Net-(D22-Pad2)
- SW23 pad 2: Net-(D22-Pad2) -> Net-(D23-Pad2)
- SW24 pad 1: L-col4 -> L-col5
- SW24 pad 2: Net-(D23-Pad2) -> Net-(D24-Pad2)
- SW25 pad 1: L-col5 -> L-col6
- SW25 pad 2: Net-(D24-Pad2) -> Net-(D25-Pad2)
- SW26 pad 1: L-col5 -> L-col4
- SW26 pad 2: Net-(D25-Pad2) -> Net-(D26-Pad2)
- SW27 pad 2: Net-(D26-Pad2) -> Net-(D27-Pad2)
- SW28 pad 1: L-col5 -> L-col6
- SW28 pad 2: Net-(D27-Pad2) -> Net-(D28-Pad2)
- SW29 pad 1: L-col5 -> R-col0
- SW29 pad 2: Net-(D28-Pad2) -> Net-(D29-Pad2)
- SW3 pad 1: L-col0 -> L-col2
- SW30 pad 1: R-col0 -> R-col1
- SW30 pad 2: Net-(D29-Pad2) -> Net-(D30-Pad2)
- SW31 pad 1: R-col1 -> R-col2
- SW31 pad 2: Net-(D30-Pad2) -> Net-(D31-Pad2)
- SW32 pad 1: R-col1 -> R-col3
- SW32 pad 2: Net-(D31-Pad2) -> Net-(D32-Pad2)
- SW33 pad 1: R-col2 -> R-col4
- SW33 pad 2: Net-(D32-Pad2) -> Net-(D33-Pad2)
- SW34 pad 1: R-col2 -> R-col5
- SW34 pad 2: Net-(D33-Pad2) -> Net-(D34-Pad2)
- SW35 pad 1: R-col2 -> R-col6
- SW35 pad 2: Net-(D34-Pad2) -> Net-(D35-Pad2)
- SW36 pad 1: R-col2 -> R-col7
- SW36 pad 2: Net-(D35-Pad2) -> Net-(D36-Pad2)
- SW37 pad 1: R-col2 -> R-col8
- SW37 pad 2: Net-(D36-Pad2) -> Net-(D37-Pad2)
- SW38 pad 1: R-col3 -> R-col0
- SW38 pad 2: Net-(D37-Pad2) -> Net-(D38-Pad2)
- SW39 pad 1: R-col3 -> R-col1
- SW39 pad 2: Net-(D38-Pad2) -> Net-(D39-Pad2)
- SW4 pad 1: L-col0 -> L-col3
- SW40 pad 1: R-col3 -> R-col2
- SW40 pad 2: Net-(D39-Pad2) -> Net-(D40-Pad2)
- SW41 pad 2: Net-(D40-Pad2) -> Net-(D41-Pad2)
- SW42 pad 1: R-col3 -> R-col4
- SW42 pad 2: Net-(D41-Pad2) -> Net-(D42-Pad2)
- SW43 pad 1: R-col4 -> R-col5
- SW43 pad 2: Net-(D42-Pad2) -> Net-(D43-Pad2)
- SW44 pad 1: R-col4 -> R-col6
- SW44 pad 2: Net-(D43-Pad2) -> Net-(D44-Pad2)
- SW45 pad 1: R-col4 -> R-col7
- SW45 pad 2: Net-(D44-Pad2) -> Net-(D45-Pad2)
- SW46 pad 1: R-col4 -> R-col8
- SW46 pad 2: Net-(D45-Pad2) -> Net-(D46-Pad2)
- SW47 pad 1: R-col4 -> R-col1
- SW47 pad 2: Net-(D46-Pad2) -> Net-(D47-Pad2)
- SW48 pad 1: R-col5 -> R-col2
- SW48 pad 2: Net-(D47-Pad2) -> Net-(D48-Pad2)
- SW49 pad 1: R-col5 -> R-col3
- SW49 pad 2: Net-(D48-Pad2) -> Net-(D49-Pad2)
- SW5 pad 1: L-col1 -> L-col4
- SW50 pad 1: R-col5 -> R-col4
- SW50 pad 2: Net-(D49-Pad2) -> Net-(D50-Pad2)
- SW51 pad 2: Net-(D50-Pad2) -> Net-(D51-Pad2)
- SW52 pad 2: Net-(D51-Pad2) -> Net-(D52-Pad2)
- SW53 pad 1: R-col6 -> R-col7
- SW53 pad 2: Net-(D52-Pad2) -> Net-(D53-Pad2)
- SW54 pad 1: R-col6 -> R-col8
- SW54 pad 2: Net-(D53-Pad2) -> Net-(D54-Pad2)
- SW55 pad 1: R-col6 -> R-col1
- SW55 pad 2: Net-(D54-Pad2) -> Net-(D55-Pad2)
- SW56 pad 1: R-col7 -> R-col2
- SW56 pad 2: Net-(D55-Pad2) -> Net-(D56-Pad2)
- SW57 pad 1: R-col7 -> R-col3
- SW57 pad 2: Net-(D56-Pad2) -> Net-(D57-Pad2)
- SW58 pad 1: R-col7 -> R-col4
- SW58 pad 2: Net-(D57-Pad2) -> Net-(D58-Pad2)
- SW59 pad 1: R-col7 -> R-col5
- SW59 pad 2: Net-(D58-Pad2) -> Net-(D59-Pad2)
- SW6 pad 1: L-col1 -> L-col5
- SW60 pad 1: R-col8 -> R-col6
- SW60 pad 2: Net-(D59-Pad2) -> Net-(D60-Pad2)
- SW61 pad 1: R-col8 -> R-col7
- SW61 pad 2: Net-(D60-Pad2) -> Net-(D61-Pad2)
- SW62 pad 2: Net-(D61-Pad2) -> Net-(D62-Pad2)
- SW63 pad 1: R-col8 -> R-col1
- SW63 pad 2: Net-(D62-Pad2) -> Net-(D63-Pad2)
- SW64 pad 1: R-reset -> R-col2
- SW64 pad 2: GND -> Net-(D64-Pad2)
- SW7 pad 1: L-col1 -> L-col6
- U1 pad 14: Net-(U1-Pad14) -> L-col6

Commit message: Updated
Parts:
- moved JP3 2.57 mm to (147.9, 36.9), turned to 180 degrees
Routing:
- net GND: track 0.00 -> 545.9 mm, vias 0 -> 30
- net VCC: track 0.00 -> 428.9 mm, vias 0 -> 6
- net R-row4: track 0.00 -> 289.5 mm, vias 0 -> 2
- net R-row3: track 0.00 -> 265.3 mm, vias 0 -> 3
- net R-col1: track 0.00 -> 245.8 mm, vias 0 -> 5
- net R-row1: track 0.00 -> 242.5 mm, vias 0 -> 3
- net R-row2: track 0.00 -> 235.4 mm, vias 0 -> 3
- net R-row0: track 0.00 -> 221.2 mm, vias 0 -> 3
- net L-row3: track 0.00 -> 219.3 mm, vias 0 -> 3
- net L-col5: track 0.00 -> 213.9 mm, vias 0 -> 4
- net R-data: track 0.00 -> 208.2 mm
- net R-col2: track 0.00 -> 198.3 mm, vias 0 -> 4
- net L-col4: track 0.00 -> 196.5 mm, vias 0 -> 5
- net L-col6: track 0.00 -> 194.2 mm
- net R-col3: track 0.00 -> 189.5 mm, vias 0 -> 3
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- added copper zone on B.Cu, net GND
- added copper zone on F.Cu, net GND

Commit message: updated
Routing:
- net GND: vias 30 -> 29
Other:
- board outline added: 305 x 95.4 mm
Changed lines of the file:
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@@
   (general
     (thickness 1.6)
-    (drawings 440)
-    (tracks 1606)
+    (drawings 448)
+    (tracks 1605)
     (zones 0)
     (modules 153)
@@
   )
   (setup
-    (last_trace_width 0.5)
+    (last_trace_width 0.25)
     (user_trace_width 0.5)
     (trace_clearance 0.2)
@@
   )
   (module MX_Alps_Hybrid:MX-1U-NoLED (layer F.Cu)
+    (at 134.895084 48.9826)
+    (fp_text reference SW13 (at 0 3.175) (layer F.SilkS)
+      (effects (font (size 1 1) (thickness 0.15)))
+    )
+    (fp_text value SW_PUSH (at 0 -7.9375) (layer F.SilkS)
+      (effects (font (size 1 1) (thickness 0.15)))
+    )
+    (fp_line (start -9.525 9.525) (end -9.525 -9.525) (layer Dwgs.User) (width 0.15))
+    (fp_line (start 9.525 9.525) (end -9.525 9.525) (layer Dwgs.User) (width 0.15))
+    (fp_line (start 9.525 -9.525) (end 9.525 9.525) (layer Dwgs.User) (width 0.15))
+    (fp_line (start -9.525 -9.525) (end 9.525 -9.525) (layer Dwgs.User) (width 0.15))
+    (fp_line (start -7 -7) (end -7 -5) (layer F.SilkS) (width 0.15))
+    (fp_line (start -5 -7) (end -7 -7) (layer F.SilkS) (width 0.15))
+    (fp_line (start -7 7) (end -5 7) (layer F.SilkS) (width 0.15))
+    (fp_line (start -7 5) (end -7 7) (layer F.SilkS) (width 0.15))
+    (fp_line (start 7 7) (end 7 5) (layer F.SilkS) (width 0.15))
+    (fp_line (start 5 7) (end 7 7) (layer F.SilkS) (width 0.15))
+    (fp_line (start 7 -7) (end 7 -5) (layer F.SilkS) (width 0.15))
+    (fp_line (start 5 -7) (end 7 -7) (layer F.SilkS) (width 0.15))
+    (pad "" np_thru_hole circle (at 5.08 0 48.0996) (size 1.75 1.75) (drill 1.75) (layers *.Cu *.Mask))
+    (pad "" np_thru_hole circle (at -5.08 0 48.0996) (size 1.75 1.75) (drill 1.75) (layers *.Cu *.Mask))
+    (pad 1 thru_hole circle (at -2.5 -4) (size 2.25 2.25) (drill 1.47) (layers *.Cu B.Mask)
+      (net 96 L-col6))
+    (pad "" np_thru_hole circle (at 0 0) (size 3.9878 3.9878) (drill 3.9878) (layers *.Cu *.Mask))
+    (pad 1 thru_hole oval (at -3.81 -2.54 48.0996) (size 4.211556 2.25) (drill 1.47 (offset 0.980778 0)) (layers *.Cu B.Mask)
+      (net 96 L-col6))
+    (pad 2 thru_hole circle (at 2.54 -5.08) (size 2.25 2.25) (drill 1.47) (layers *.Cu B.Mask)
+      (net 15 "Net-(D13-Pad2)"))
+    (pad 2 thru_hole oval (at 2.5 -4.5 86.0548) (size 2.831378 2.25) (drill 1.47 (offset 0.290689 0)) (layers *.Cu B.Mask)
+      (net 15 "Net-(D13-Pad2)"))
+  )
+  (module MX_Alps_Hybrid:MX-1U-NoLED (layer F.Cu)
     (at 58.695084 48.9826)
     (fp_text reference SW9 (at 0 3.175) (layer F.SilkS)
@@
   )
   (module MX_Alps_Hybrid:MX-1U-NoLED (layer F.Cu)
-    (at 134.895084 48.9826)
-    (fp_text reference SW13 (at 0 3.175) (layer F.SilkS)
-      (effects (font (size 1 1) (thickness 0.15)))
-    )
-    (fp_text value SW_PUSH (at 0 -7.9375) (layer F.SilkS)
-      (effects (font (size 1 1) (thickness 0.15)))
-    )
-    (fp_line (start -9.525 9.525) (end -9.525 -9.525) (layer Dwgs.User) (width 0.15))
-    (fp_line (start 9.525 9.525) (end -9.525 9.525) (layer Dwgs.User) (width 0.15))
-    (fp_line (start 9.525 -9.525) (end 9.525 9.525) (layer Dwgs.User) (width 0.15))
-    (fp_line (start -9.525 -9.525) (end 9.525 -9.525) (layer Dwgs.User) (width 0.15))
-    (fp_line (start -7 -7) (end -7 -5) (layer F.SilkS) (width 0.15))
-    (fp_line (start -5 -7) (end -7 -7) (layer F.SilkS) (width 0.15))
-    (fp_line (start -7 7) (end -5 7) (layer F.SilkS) (width 0.15))
-    (fp_line (start -7 5) (end -7 7) (layer F.SilkS) (width 0.15))
-    (fp_line (start 7 7) (end 7 5) (layer F.SilkS) (width 0.15))
-    (fp_line (start 5 7) (end 7 7) (layer F.SilkS) (width 0.15))
-    (fp_line (start 7 -7) (end 7 -5) (layer F.SilkS) (width 0.15))
-    (fp_line (start 5 -7) (end 7 -7) (layer F.SilkS) (width 0.15))
-    (pad "" np_thru_hole circle (at 5.08 0 48.0996) (size 1.75 1.75) (drill 1.75) (layers *.Cu *.Mask))
-    (pad "" np_thru_hole circle (at -5.08 0 48.0996) (size 1.75 1.75) (drill 1.75) (layers *.Cu *.Mask))
-    (pad 1 thru_hole circle (at -2.5 -4) (size 2.25 2.25) (drill 1.47) (layers *.Cu B.Mask)
-      (net 96 L-col6))
-    (pad "" np_thru_hole circle (at 0 0) (size 3.9878 3.9878) (drill 3.9878) (layers *.Cu *.Mask))
-    (pad 1 thru_hole oval (at -3.81 -2.54 48.0996) (size 4.211556 2.25) (drill 1.47 (offset 0.980778 0)) (layers *.Cu B.Mask)
-      (net 96 L-col6))
-    (pad 2 thru_hole circle (at 2.54 -5.08) (size 2.25 2.25) (drill 1.47) (layers *.Cu B.Mask)
-      (net 15 "Net-(D13-Pad2)"))
-    (pad 2 thru_hole oval (at 2.5 -4.5 86.0548) (size 2.831378 2.25) (drill 1.47 (offset 0.290689 0)) (layers *.Cu B.Mask)
-      (net 15 "Net-(D13-Pad2)"))
-  )
-  (module MX_Alps_Hybrid:MX-1U-NoLED (layer F.Cu)
     (at 63.457584 68.0326)
     (fp_text reference SW15 (at 0 3.175) (layer F.SilkS)
@@
       (net 87 R-led))
   )
+  (gr_line (start 149.105084 115.7576) (end 149.265084 115.7576) (layer Edge.Cuts) (width 0.05))
+  (gr_line (start 153.145084 20.3076) (end 154.755084 20.3076) (layer Edge.Cuts) (width 0.05))
+  (gr_line (start 325.495084 20.3076) (end 154.755084 20.3076) (layer Edge.Cuts) (width 0.05))
+  (gr_line (start 149.265084 115.7576) (end 325.495084 115.7576) (layer Edge.Cuts) (width 0.05))
+  (gr_line (start 149.105084 115.7576) (end 20.495084 115.7576) (layer Edge.Cuts) (width 0.05))
+  (gr_line (start 153.145084 20.3076) (end 20.495084 20.3076) (layer Edge.Cuts) (width 0.05))
+  (gr_line (start 20.495084 115.7576) (end 20.495084 20.3076) (layer Edge.Cuts) (width 0.05))
+  (gr_line (start 325.495084 20.3076) (end 325.495084 115.7576) (layer Edge.Cuts) (width 0.05))
   (gr_line (start 308.87 36.931701) (end 308.87 22.9324) (layer Dwgs.User) (width 0.2))
   (gr_line (start 322.869 36.931701) (end 308.87 36.931701) (layer Dwgs.User) (width 0.2))
@@
   (via (at 128.645084 37.5576) (size 0.8) (drill 0.4) (layers F.Cu B.Cu) (net 82))
   (via (at 87.445084 35.4576) (size 0.8) (drill 0.4) (layers F.Cu B.Cu) (net 82))
-  (via (at 280.895084 33.3076) (size 0.8) (drill 0.4) (layers F.Cu B.Cu) (net 82))
   (via (at 186.445084 39.1076) (size 0.8) (drill 0.4) (layers F.Cu B.Cu) (net 82))
   (via (at 243.195084 34.6576) (size 0.8) (drill 0.4) (layers F.Cu B.Cu) (net 82))
@@
   (via (at 222.295084 34.5576) (size 0.8) (drill 0.4) (layers F.Cu B.Cu) (net 82))
   (via (at 204.745084 34.5576) (size 0.8) (drill 0.4) (layers F.Cu B.Cu) (net 82))
-  (via (at 322.145084 26.0076) (size 0.8) (drill 0.4) (layers F.Cu B.Cu) (net 82))
   (via (at 112.295084 35.3076) (size 0.8) (drill 0.4) (layers F.Cu B.Cu) (net 82))
   (via (at 69.595084 36.2576) (size 0.8) (drill 0.4) (layers F.Cu B.Cu) (net 82))
@@
   (segment (start 318.745084 85.9076) (end 316.395084 83.5576) (width 0.5) (layer F.Cu) (net 82))
   (segment (start 312.445084 89.7576) (end 317.195084 89.7576) (width 0.5) (layer F.Cu) (net 82))
+  (via (at 272.395084 34.1376) (size 0.8) (drill 0.4) (layers F.Cu B.Cu) (net 82))
   (segment (start 22.195084 44.40798) (end 22.195084 46.6076) (width 0.25) (layer F.Cu) (net 83))
   (segment (start 29.920302 40.2076) (end 38.845084 40.2076) (width 0.25) (layer F.Cu) (net 83))
