File: iroha60/pcb/iroha60-left/iroha60-left.sch (KiCad schematic (older format))
At the start: 63 parts, among them J1 i2c-pin, J2 MJ-4PP-9, J3 i2c-pin, J4 LED, SW1 SW_PUSH, SW10 SW_PUSH, SW11 SW_PUSH, SW12 SW_PUSH, SW13 SW_PUSH, SW14 SW_PUSH, SW15 SW_PUSH, SW16 SW_PUSH, SW17 SW_PUSH, SW18 SW_PUSH, SW19 SW_PUSH, SW2 SW_PUSH, SW20 SW_PUSH, SW21 SW_PUSH, SW22 SW_PUSH, SW23 SW_PUSH, SW24 SW_PUSH, SW25 SW_PUSH, SW26 SW_PUSH, SW27 SW_PUSH, SW28 SW_PUSH, SW29 RESET_SW, SW3 SW_PUSH, SW4 SW_PUSH, SW5 SW_PUSH, SW6 SW_PUSH, SW7 SW_PUSH, SW8 SW_PUSH, SW9 SW_PUSH, U1 ProMicro

Commit message: PCB Updated
Parts:
- D1, D10, D11, D12, D13, D14, D15, D16, D17, D18, D19, D2, D20, D21, D22, D23, D24, D25, D26, D27, D28, D3, D4, D5, D6, D7, D8, D9: footprint (none) -> kbd:D3_TH_SMD
- J1, J3: footprint (none) -> kbd:1pin_conn
- J2: footprint (none) -> kbd:MJ-4PP-9_1side
- J4: footprint (none) -> kbd:StripLED_1side
- JP1: footprint (none) -> kbd:Jumper
- SW1, SW10, SW11, SW12, SW13, SW15, SW16, SW17, SW18, SW19, SW2, SW21, SW22, SW23, SW24, SW25, SW26, SW3, SW4, SW5, SW6, SW7, SW9: footprint (none) -> MX_Alps_Hybrid:MX-1U-NoLED
- SW14: footprint (none) -> MX_Alps_Hybrid:MX-1.75U-NoLED
- SW20: footprint (none) -> MX_Alps_Hybrid:MX-2.25U-ReversedStabilizers-NoLED
- SW27, SW8: footprint (none) -> MX_Alps_Hybrid:MX-1.5U-NoLED
- SW28: footprint (none) -> MX_Alps_Hybrid:MX-2.75U-ReversedStabilizers-NoLED
- SW29: footprint (none) -> kbd:ResetSW_1side
- U1: footprint (none) -> kbd:ProMicro_v3.5

Commit message: Updated
Parts:
- U1: footprint kbd:ProMicro_v3.5 -> kbd:ProMicro_v3
Changed lines of the file:
@@
 F 0 "U1" H 1975 7137 60  0000 C CNN
 F 1 "ProMicro" H 1975 7031 60  0000 C CNN
-F 2 "kbd:ProMicro_v3.5" H 2075 5050 60  0001 C CNN
+F 2 "kbd:ProMicro_v3" H 2075 5050 60  0001 C CNN
 F 3 "" H 2075 5050 60  0000 C CNN
 	1    1975 6100

Commit message: Updated
Parts:
- SW1, SW10, SW11, SW12, SW13, SW15, SW16, SW17, SW18, SW19, SW2, SW21, SW22, SW23, SW24, SW25, SW26, SW3, SW4, SW5, SW6, SW7, SW9: footprint MX_Alps_Hybrid:MX-1U-NoLED -> keyswitches:Kailh_socket_MX_optional
- SW14: footprint MX_Alps_Hybrid:MX-1.75U-NoLED -> keyswitches:Kailh_socket_MX_optional
- SW20: footprint MX_Alps_Hybrid:MX-2.25U-ReversedStabilizers-NoLED -> keyswitches:Kailh_socket_MX_optional
- SW27, SW8: footprint MX_Alps_Hybrid:MX-1.5U-NoLED -> keyswitches:Kailh_socket_MX_optional
- SW28: footprint MX_Alps_Hybrid:MX-2.75U-ReversedStabilizers-NoLED -> keyswitches:Kailh_socket_MX_optional
Changed lines of the file:
@@
 F 0 "SW1" H 3325 1605 50  0000 C CNN
 F 1 "SW_PUSH" H 3325 1514 50  0000 C CNN
-F 2 "MX_Alps_Hybrid:MX-1U-NoLED" H 3325 1350 50  0001 C CNN
+F 2 "keyswitches:Kailh_socket_MX_optional" H 3325 1350 50  0001 C CNN
 F 3 "" H 3325 1350 50  0000 C CNN
 	1    3325 1350
@@
 F 0 "SW2" H 4175 1605 50  0000 C CNN
 F 1 "SW_PUSH" H 4175 1514 50  0000 C CNN
-F 2 "MX_Alps_Hybrid:MX-1U-NoLED" H 4175 1350 50  0001 C CNN
+F 2 "keyswitches:Kailh_socket_MX_optional" H 4175 1350 50  0001 C CNN
 F 3 "" H 4175 1350 50  0000 C CNN
 	1    4175 1350
@@
 F 0 "SW3" H 5050 1605 50  0000 C CNN
 F 1 "SW_PUSH" H 5050 1514 50  0000 C CNN
-F 2 "MX_Alps_Hybrid:MX-1U-NoLED" H 5050 1350 50  0001 C CNN
+F 2 "keyswitches:Kailh_socket_MX_optional" H 5050 1350 50  0001 C CNN
 F 3 "" H 5050 1350 50  0000 C CNN
 	1    5050 1350
@@
 F 0 "SW4" H 5900 1605 50  0000 C CNN
 F 1 "SW_PUSH" H 5900 1514 50  0000 C CNN
-F 2 "MX_Alps_Hybrid:MX-1U-NoLED" H 5900 1350 50  0001 C CNN
+F 2 "keyswitches:Kailh_socket_MX_optional" H 5900 1350 50  0001 C CNN
 F 3 "" H 5900 1350 50  0000 C CNN
 	1    5900 1350
@@
 F 0 "SW5" H 6750 1605 50  0000 C CNN
 F 1 "SW_PUSH" H 6750 1514 50  0000 C CNN
-F 2 "MX_Alps_Hybrid:MX-1U-NoLED" H 6750 1350 50  0001 C CNN
+F 2 "keyswitches:Kailh_socket_MX_optional" H 6750 1350 50  0001 C CNN
 F 3 "" H 6750 1350 50  0000 C CNN
 	1    6750 1350
@@
 F 0 "SW6" H 7600 1605 50  0000 C CNN
 F 1 "SW_PUSH" H 7600 1514 50  0000 C CNN
-F 2 "MX_Alps_Hybrid:MX-1U-NoLED" H 7600 1350 50  0001 C CNN
+F 2 "keyswitches:Kailh_socket_MX_optional" H 7600 1350 50  0001 C CNN
 F 3 "" H 7600 1350 50  0000 C CNN
 	1    7600 1350
@@
 F 0 "SW7" H 8475 1605 50  0000 C CNN
 F 1 "SW_PUSH" H 8475 1514 50  0000 C CNN
-F 2 "MX_Alps_Hybrid:MX-1U-NoLED" H 8475 1350 50  0001 C CNN
+F 2 "keyswitches:Kailh_socket_MX_optional" H 8475 1350 50  0001 C CNN
 F 3 "" H 8475 1350 50  0000 C CNN
 	1    8475 1350
@@
 F 0 "SW9" H 5050 2330 50  0000 C CNN
 F 1 "SW_PUSH" H 5050 2239 50  0000 C CNN
-F 2 "MX_Alps_Hybrid:MX-1U-NoLED" H 5050 2075 50  0001 C CNN
+F 2 "keyswitches:Kailh_socket_MX_optional" H 5050 2075 50  0001 C CNN
 F 3 "" H 5050 2075 50  0000 C CNN
 	1    5050 2075
@@
 F 0 "SW10" H 5900 2330 50  0000 C CNN
 F 1 "SW_PUSH" H 5900 2239 50  0000 C CNN
-F 2 "MX_Alps_Hybrid:MX-1U-NoLED" H 5900 2075 50  0001 C CNN
+F 2 "keyswitches:Kailh_socket_MX_optional" H 5900 2075 50  0001 C CNN
 F 3 "" H 5900 2075 50  0000 C CNN
 	1    5900 2075
@@
 F 0 "SW11" H 6750 2330 50  0000 C CNN
 F 1 "SW_PUSH" H 6750 2239 50  0000 C CNN
-F 2 "MX_Alps_Hybrid:MX-1U-NoLED" H 6750 2075 50  0001 C CNN
+F 2 "keyswitches:Kailh_socket_MX_optional" H 6750 2075 50  0001 C CNN
 F 3 "" H 6750 2075 50  0000 C CNN
 	1    6750 2075
@@
 F 0 "SW12" H 7600 2330 50  0000 C CNN
 F 1 "SW_PUSH" H 7600 2239 50  0000 C CNN
-F 2 "MX_Alps_Hybrid:MX-1U-NoLED" H 7600 2075 50  0001 C CNN
+F 2 "keyswitches:Kailh_socket_MX_optional" H 7600 2075 50  0001 C CNN
 F 3 "" H 7600 2075 50  0000 C CNN
 	1    7600 2075
@@
 F 0 "SW13" H 8475 2330 50  0000 C CNN
 F 1 "SW_PUSH" H 8475 2239 50  0000 C CNN
-F 2 "MX_Alps_Hybrid:MX-1U-NoLED" H 8475 2075 50  0001 C CNN
+F 2 "keyswitches:Kailh_socket_MX_optional" H 8475 2075 50  0001 C CNN
 F 3 "" H 8475 2075 50  0000 C CNN
 	1    8475 2075
@@
 F 0 "SW15" H 5050 3030 50  0000 C CNN
 F 1 "SW_PUSH" H 5050 2939 50  0000 C CNN
-F 2 "MX_Alps_Hybrid:MX-1U-NoLED" H 5050 2775 50  0001 C CNN
+F 2 "keyswitches:Kailh_socket_MX_optional" H 5050 2775 50  0001 C CNN
 F 3 "" H 5050 2775 50  0000 C CNN
 	1    5050 2775
@@
 F 0 "SW16" H 5900 3030 50  0000 C CNN
 F 1 "SW_PUSH" H 5900 2939 50  0000 C CNN
-F 2 "MX_Alps_Hybrid:MX-1U-NoLED" H 5900 2775 50  0001 C CNN
+F 2 "keyswitches:Kailh_socket_MX_optional" H 5900 2775 50  0001 C CNN
 F 3 "" H 5900 2775 50  0000 C CNN
 	1    5900 2775
@@
 F 0 "SW17" H 6750 3030 50  0000 C CNN
 F 1 "SW_PUSH" H 6750 2939 50  0000 C CNN
-F 2 "MX_Alps_Hybrid:MX-1U-NoLED" H 6750 2775 50  0001 C CNN
+F 2 "keyswitches:Kailh_socket_MX_optional" H 6750 2775 50  0001 C CNN
 F 3 "" H 6750 2775 50  0000 C CNN
 	1    6750 2775
@@
 F 0 "SW18" H 7600 3030 50  0000 C CNN
 F 1 "SW_PUSH" H 7600 2939 50  0000 C CNN
-F 2 "MX_Alps_Hybrid:MX-1U-NoLED" H 7600 2775 50  0001 C CNN
+F 2 "keyswitches:Kailh_socket_MX_optional" H 7600 2775 50  0001 C CNN
 F 3 "" H 7600 2775 50  0000 C CNN
 	1    7600 2775
@@
 F 0 "SW19" H 8475 3030 50  0000 C CNN
 F 1 "SW_PUSH" H 8475 2939 50  0000 C CNN
-F 2 "MX_Alps_Hybrid:MX-1U-NoLED" H 8475 2775 50  0001 C CNN
+F 2 "keyswitches:Kailh_socket_MX_optional" H 8475 2775 50  0001 C CNN
 F 3 "" H 8475 2775 50  0000 C CNN
 	1    8475 2775
@@
 F 0 "SW21" H 5050 3755 50  0000 C CNN
 F 1 "SW_PUSH" H 5050 3664 50  0000 C CNN
-F 2 "MX_Alps_Hybrid:MX-1U-NoLED" H 5050 3500 50  0001 C CNN
+F 2 "keyswitches:Kailh_socket_MX_optional" H 5050 3500 50  0001 C CNN
 F 3 "" H 5050 3500 50  0000 C CNN
 	1    5050 3500
@@
 F 0 "SW22" H 5900 3755 50  0000 C CNN
 F 1 "SW_PUSH" H 5900 3664 50  0000 C CNN
-F 2 "MX_Alps_Hybrid:MX-1U-NoLED" H 5900 3500 50  0001 C CNN
+F 2 "keyswitches:Kailh_socket_MX_optional" H 5900 3500 50  0001 C CNN
 F 3 "" H 5900 3500 50  0000 C CNN
 	1    5900 3500
@@
 F 0 "SW23" H 6750 3755 50  0000 C CNN
 F 1 "SW_PUSH" H 6750 3664 50  0000 C CNN
-F 2 "MX_Alps_Hybrid:MX-1U-NoLED" H 6750 3500 50  0001 C CNN
+F 2 "keyswitches:Kailh_socket_MX_optional" H 6750 3500 50  0001 C CNN
 F 3 "" H 6750 3500 50  0000 C CNN
 	1    6750 3500
@@
 F 0 "SW24" H 7600 3755 50  0000 C CNN
 F 1 "SW_PUSH" H 7600 3664 50  0000 C CNN
-F 2 "MX_Alps_Hybrid:MX-1U-NoLED" H 7600 3500 50  0001 C CNN
+F 2 "keyswitches:Kailh_socket_MX_optional" H 7600 3500 50  0001 C CNN
 F 3 "" H 7600 3500 50  0000 C CNN
 	1    7600 3500
@@
 F 0 "SW25" H 8475 3755 50  0000 C CNN
 F 1 "SW_PUSH" H 8475 3664 50  0000 C CNN
-F 2 "MX_Alps_Hybrid:MX-1U-NoLED" H 8475 3500 50  0001 C CNN
+F 2 "keyswitches:Kailh_socket_MX_optional" H 8475 3500 50  0001 C CNN
 F 3 "" H 8475 3500 50  0000 C CNN
 	1    8475 3500
@@
 F 0 "SW26" H 6750 4480 50  0000 C CNN
 F 1 "SW_PUSH" H 6750 4389 50  0000 C CNN
-F 2 "MX_Alps_Hybrid:MX-1U-NoLED" H 6750 4225 50  0001 C CNN
+F 2 "keyswitches:Kailh_socket_MX_optional" H 6750 4225 50  0001 C CNN
 F 3 "" H 6750 4225 50  0000 C CNN
 	1    6750 4225
@@
 F 0 "SW27" H 7600 4480 50  0000 C CNN
 F 1 "SW_PUSH" H 7600 4389 50  0000 C CNN
-F 2 "MX_Alps_Hybrid:MX-1.5U-NoLED" H 7600 4225 50  0001 C CNN
+F 2 "keyswitches:Kailh_socket_MX_optional" H 7600 4225 50  0001 C CNN
 F 3 "" H 7600 4225 50  0000 C CNN
 	1    7600 4225
@@
 F 0 "SW28" H 8475 4480 50  0000 C CNN
 F 1 "SW_PUSH" H 8475 4389 50  0000 C CNN
-F 2 "MX_Alps_Hybrid:MX-2.75U-ReversedStabilizers-NoLED" H 8475 4225 50  0001 C CNN
+F 2 "keyswitches:Kailh_socket_MX_optional" H 8475 4225 50  0001 C CNN
 F 3 "" H 8475 4225 50  0000 C CNN
 	1    8475 4225
@@
 F 0 "SW20" H 4175 3755 50  0000 C CNN
 F 1 "SW_PUSH" H 4175 3664 50  0000 C CNN
-F 2 "MX_Alps_Hybrid:MX-2.25U-ReversedStabilizers-NoLED" H 4175 3500 50  0001 C CNN
+F 2 "keyswitches:Kailh_socket_MX_optional" H 4175 3500 50  0001 C CNN
 F 3 "" H 4175 3500 50  0000 C CNN
 	1    4175 3500
@@
 F 0 "SW14" H 4175 3030 50  0000 C CNN
 F 1 "SW_PUSH" H 4175 2939 50  0000 C CNN
-F 2 "MX_Alps_Hybrid:MX-1.75U-NoLED" H 4175 2775 50  0001 C CNN
+F 2 "keyswitches:Kailh_socket_MX_optional" H 4175 2775 50  0001 C CNN
 F 3 "" H 4175 2775 50  0000 C CNN
 	1    4175 2775
@@
 F 0 "SW8" H 4175 2330 50  0000 C CNN
 F 1 "SW_PUSH" H 4175 2239 50  0000 C CNN
-F 2 "MX_Alps_Hybrid:MX-1.5U-NoLED" H 4175 2075 50  0001 C CNN
+F 2 "keyswitches:Kailh_socket_MX_optional" H 4175 2075 50  0001 C CNN
 F 3 "" H 4175 2075 50  0000 C CNN
 	1    4175 2075

Commit message: Updated
Parts:
- added J3: Conn_01x04, kbd:OLED_1side, symbol Connector_Generic:Conn_01x04
- added JP1, JP2, JP3, JP5: Jumper_NO_Small, kbd:Jumper, symbol Device:Jumper_NO_Small
- added R1, R2: R, Resistor_THT:R_Axial_DIN0204_L3.6mm_D1.6mm_P5.08mm_Horizontal, symbol Device:R
- renumbered J3 to J4, J4 to J5, JP1 to JP4
Connections:
- net GND: now also JP1.2
- net VCC: now also JP2.2, R1.1, R2.1
- net SDA: now reaches U1.5 (2/D1/SDA)
- net SDA: now also JP5.2, R1.2
- net SCL: now reaches U1.6 (3/D0/SCL)
- net SCL: now also JP3.2, R2.2
- new net: J3.1 (Pin_1), JP5.1
- new net: J3.2 (Pin_2), JP3.1
- new net: J3.3 (Pin_3), JP2.1
- new net: J3.4 (Pin_4), JP1.1
- no-connect marks 5 -> 3
Changed lines of the file:
@@
 $EndComp
 $Comp
-L power:GND #PWR06
+L power:GND #PWR08
 U 1 1 5E04F284
 P 3300 5500
-F 0 "#PWR06" H 3300 5250 50  0001 C CNN
+F 0 "#PWR08" H 3300 5250 50  0001 C CNN
 F 1 "GND" H 3305 5327 50  0000 C CNN
 F 2 "" H 3300 5500 50  0001 C CNN
@@
 $EndComp
 $Comp
-L power:GND #PWR08
+L power:GND #PWR010
 U 1 1 5E050AF8
 P 925 5725
-F 0 "#PWR08" H 925 5475 50  0001 C CNN
+F 0 "#PWR010" H 925 5475 50  0001 C CNN
 F 1 "GND" H 930 5552 50  0000 C CNN
 F 2 "" H 925 5725 50  0001 C CNN
@@
 Text GLabel 2675 6350 2    50   Input ~ 0
 col6
-NoConn ~ 1275 5750
-NoConn ~ 1275 5850
 NoConn ~ 1275 6450
 NoConn ~ 2675 5350
@@
 $EndComp
 $Comp
-L Device:Jumper JP1
+L Device:Jumper JP4
 U 1 1 5E053848
 P 7250 5550
-F 0 "JP1" H 7250 5325 50  0000 C CNN
+F 0 "JP4" H 7250 5325 50  0000 C CNN
 F 1 "Jumper" H 7250 5416 50  0000 C CNN
 F 2 "kbd:Jumper" H 7250 5550 50  0001 C CNN
@@
 $EndComp
 $Comp
-L power:VCC #PWR04
+L power:VCC #PWR05
 U 1 1 5E05495B
 P 6400 5300
-F 0 "#PWR04" H 6400 5150 50  0001 C CNN
+F 0 "#PWR05" H 6400 5150 50  0001 C CNN
 F 1 "VCC" H 6417 5473 50  0000 C CNN
 F 2 "" H 6400 5300 50  0001 C CNN
@@
 $EndComp
 $Comp
-L power:GND #PWR07
+L power:GND #PWR09
 U 1 1 5E05507C
 P 6400 5600
-F 0 "#PWR07" H 6400 5350 50  0001 C CNN
+F 0 "#PWR09" H 6400 5350 50  0001 C CNN
 F 1 "GND" H 6405 5427 50  0000 C CNN
 F 2 "" H 6400 5600 50  0001 C CNN
@@
 $EndComp
 $Comp
-L Connector_Generic:Conn_01x01 J3
+L Connector_Generic:Conn_01x01 J4
 U 1 1 5E057B6E
 P 6775 5925
-F 0 "J3" V 6647 6005 50  0000 L CNN
+F 0 "J4" V 6647 6005 50  0000 L CNN
 F 1 "i2c-pin" V 6738 6005 50  0000 L CNN
 F 2 "kbd:1pin_conn" H 6775 5925 50  0001 C CNN
@@
 $EndComp
 $Comp
-L Connector_Generic:Conn_01x03 J4
+L Connector_Generic:Conn_01x03 J5
 U 1 1 5E05841F
 P 4150 6450
-F 0 "J4" H 4068 6125 50  0000 C CNN
+F 0 "J5" H 4068 6125 50  0000 C CNN
 F 1 "LED" H 4068 6216 50  0000 C CNN
 F 2 "kbd:StripLED_1side" H 4150 6450 50  0001 C CNN
@@
 $EndComp
 $Comp
-L power:VCC #PWR09
+L power:VCC #PWR013
 U 1 1 5E059132
 P 4675 6300
-F 0 "#PWR09" H 4675 6150 50  0001 C CNN
+F 0 "#PWR013" H 4675 6150 50  0001 C CNN
 F 1 "VCC" H 4692 6473 50  0000 C CNN
 F 2 "" H 4675 6300 50  0001 C CNN
@@
 $EndComp
 $Comp
-L power:GND #PWR010
+L power:GND #PWR014
 U 1 1 5E05980D
 P 4675 6600
-F 0 "#PWR010" H 4675 6350 50  0001 C CNN
+F 0 "#PWR014" H 4675 6350 50  0001 C CNN
 F 1 "GND" H 4680 6427 50  0000 C CNN
 F 2 "" H 4675 6600 50  0001 C CNN
@@
 $EndComp
 $Comp
-L power:GND #PWR05
+L power:GND #PWR07
 U 1 1 5E05A732
 P 4825 5400
-F 0 "#PWR05" H 4825 5150 50  0001 C CNN
+F 0 "#PWR07" H 4825 5150 50  0001 C CNN
 F 1 "GND" H 4830 5227 50  0000 C CNN
 F 2 "" H 4825 5400 50  0001 C CNN
@@
 	8175 4225 8175 3500
 Connection ~ 8175 3500
+Text GLabel 1275 5750 0    50   Input ~ 0
+SDA
+Text GLabel 1275 5850 0    50   Input ~ 0
+SCL
+$Comp
+L Connector_Generic:Conn_01x04 J3
+U 1 1 5E9B967F
+P 8500 5475
+F 0 "J3" H 8418 5050 50  0000 C CNN
+F 1 "Conn_01x04" H 8418 5141 50  0000 C CNN
+F 2 "kbd:OLED_1side" H 8500 5475 50  0001 C CNN
+F 3 "~" H 8500 5475 50  0001 C CNN
+	1    8500 5475
+	-1   0    0    1
+$EndComp
+$Comp
+L Device:Jumper_NO_Small JP1
+U 1 1 5E9BD4A7
+P 9025 5275
+F 0 "JP1" H 9025 5460 50  0000 C CNN
+F 1 "Jumper_NO_Small" H 9025 5369 50  0000 C CNN
+F 2 "kbd:Jumper" H 9025 5275 50  0001 C CNN
+F 3 "~" H 9025 5275 50  0001 C CNN
+	1    9025 5275
+	1    0    0    -1
+$EndComp
+$Comp
+L Device:Jumper_NO_Small JP2
+U 1 1 5E9BE5E9
+P 9025 5375
+F 0 "JP2" H 9025 5560 50  0000 C CNN
+F 1 "Jumper_NO_Small" H 9025 5469 50  0000 C CNN
+F 2 "kbd:Jumper" H 9025 5375 50  0001 C CNN
+F 3 "~" H 9025 5375 50  0001 C CNN
+	1    9025 5375
+	1    0    0    -1
+$EndComp
+$Comp
+L Device:Jumper_NO_Small JP3
+U 1 1 5E9BF1DE
+P 9025 5475
+F 0 "JP3" H 9025 5660 50  0000 C CNN
+F 1 "Jumper_NO_Small" H 9025 5569 50  0000 C CNN
+F 2 "kbd:Jumper" H 9025 5475 50  0001 C CNN
+F 3 "~" H 9025 5475 50  0001 C CNN
+	1    9025 5475
+	1    0    0    -1
+$EndComp
+$Comp
+L Device:Jumper_NO_Small JP5
+U 1 1 5E9BFDE6
+P 9025 5575
+F 0 "JP5" H 9025 5760 50  0000 C CNN
+F 1 "Jumper_NO_Small" H 9025 5669 50  0000 C CNN
+F 2 "kbd:Jumper" H 9025 5575 50  0001 C CNN
+F 3 "~" H 9025 5575 50  0001 C CNN
+	1    9025 5575
+	1    0    0    -1
+$EndComp
+$Comp
+L power:GND #PWR04
+U 1 1 5E9C499F
+P 9375 5275
+F 0 "#PWR04" H 9375 5025 50  0001 C CNN
+F 1 "GND" V 9380 5147 50  0000 R CNN
+F 2 "" H 9375 5275 50  0001 C CNN
+F 3 "" H 9375 5275 50  0001 C CNN
+	1    9375 5275
+	0    -1   -1   0
+$EndComp
+$Comp
+L power:VCC #PWR06
+U 1 1 5E9C5828
+P 9375 5375
+F 0 "#PWR06" H 9375 5225 50  0001 C CNN
+F 1 "VCC" V 9392 5503 50  0000 L CNN
+F 2 "" H 9375 5375 50  0001 C CNN
+F 3 "" H 9375 5375 50  0001 C CNN
+	1    9375 5375
+	0    1    1    0
+$EndComp
+Text GLabel 9375 5575 2    50   Input ~ 0
+SDA
+Text GLabel 9375 5475 2    50   Input ~ 0
+SCL
+Wire Wire Line
+	8700 5275 8925 5275
+Wire Wire Line
+	9125 5275 9375 5275
+Wire Wire Line
+	8700 5375 8925 5375
+Wire Wire Line
+	9125 5375 9375 5375
+Wire Wire Line
+	8700 5475 8925 5475
+Wire Wire Line
+	9125 5475 9375 5475
+Wire Wire Line
+	8700 5575 8925 5575
+Wire Wire Line
+	9125 5575 9375 5575
+Text GLabel 8775 6100 0    50   Input ~ 0
+SCL
+Text GLabel 8775 5950 0    50   Input ~ 0
+SDA
+$Comp
+L Device:R R1
+U 1 1 5E9D6A10
+P 9025 5950
+F 0 "R1" V 8818 5950 50  0000 C CNN
+F 1 "R" V 8909 5950 50  0000 C CNN
+F 2 "Resistor_THT:R_Axial_DIN0204_L3.6mm_D1.6mm_P5.08mm_Horizontal" V 8955 5950 50  0001 C CNN
+F 3 "~" H 9025 5950 50  0001 C CNN
+	1    9025 5950
+	0    1    1    0
+$EndComp
+$Comp
+L Device:R R2
+U 1 1 5E9D7741
+P 9025 6100
+F 0 "R2" V 8818 6100 50  0000 C CNN
+F 1 "R" V 8909 6100 50  0000 C CNN
+F 2 "Resistor_THT:R_Axial_DIN0204_L3.6mm_D1.6mm_P5.08mm_Horizontal" V 8955 6100 50  0001 C CNN
+F 3 "~" H 9025 6100 50  0001 C CNN
+	1    9025 6100
+	0    1    1    0
+$EndComp
+$Comp
+L power:VCC #PWR011
+U 1 1 5E9D79D2
+P 9325 5950
+F 0 "#PWR011" H 9325 5800 50  0001 C CNN
+F 1 "VCC" V 9342 6078 50  0000 L CNN
+F 2 "" H 9325 5950 50  0001 C CNN
+F 3 "" H 9325 5950 50  0001 C CNN
+	1    9325 5950
+	0    1    1    0
+$EndComp
+$Comp
+L power:VCC #PWR012
+U 1 1 5E9D7FDB
+P 9325 6100
+F 0 "#PWR012" H 9325 5950 50  0001 C CNN
+F 1 "VCC" V 9342 6228 50  0000 L CNN
+F 2 "" H 9325 6100 50  0001 C CNN
+F 3 "" H 9325 6100 50  0001 C CNN
+	1    9325 6100
+	0    1    1    0
+$EndComp
+Wire Wire Line
+	8875 5950 8775 5950
+Wire Wire Line
+	9175 5950 9325 5950
+Wire Wire Line
+	9175 6100 9325 6100
+Wire Wire Line
+	8875 6100 8775 6100
 $EndSCHEMATC

Commit message: Updated
Parts:
- removed J3: Conn_01x04, kbd:OLED_1side, symbol Connector_Generic:Conn_01x04
- removed JP1, JP2, JP3, JP5: Jumper_NO_Small, kbd:Jumper, symbol Device:Jumper_NO_Small
- removed R1, R2: R, Resistor_THT:R_Axial_DIN0204_L3.6mm_D1.6mm_P5.08mm_Horizontal, symbol Device:R
- SW1, SW10, SW11, SW12, SW13, SW15, SW16, SW17, SW18, SW19, SW2, SW21, SW22, SW23, SW24, SW25, SW26, SW27, SW3, SW4, SW5, SW6, SW7, SW9: footprint keyswitches:Kailh_socket_MX_optional -> MX_Alps_Hybrid:MX-1U-NoLED
- SW14: footprint keyswitches:Kailh_socket_MX_optional -> MX_Alps_Hybrid:MX-1.75U-NoLED
- SW20: footprint keyswitches:Kailh_socket_MX_optional -> MX_Alps_Hybrid:MX-2.25U-ReversedStabilizers-NoLED
- SW28: footprint keyswitches:Kailh_socket_MX_optional -> MX_Alps_Hybrid:MX-2.75U-ReversedStabilizers-NoLED
- SW8: footprint keyswitches:Kailh_socket_MX_optional -> MX_Alps_Hybrid:MX-1.5U-NoLED
- U1: footprint kbd:ProMicro_v3 -> kbd:ProMicro_v2_1side
- renumbered J4 to J3, J5 to J4, JP4 to JP1
Connections:
- net SCL: no longer names the net of U1.6 (3/D0/SCL)
- net SDA: no longer names the net of U1.5 (2/D1/SDA)
- no-connect marks 3 -> 6

Commit message: Updated
Parts:
- removed J1, J3: i2c-pin, kbd:1pin_conn, symbol Connector_Generic:Conn_01x01
- removed JP1: Jumper, kbd:Jumper, symbol Device:Jumper
- SW27: footprint MX_Alps_Hybrid:MX-1U-NoLED -> MX_Alps_Hybrid:MX-1.5U-NoLED
Connections:
- net data: now also J2.B
Changed lines of the file:
@@
-$EndComp
-$Comp
-L Device:Jumper JP1
-U 1 1 5E053848
-P 7250 5550
-F 0 "JP1" H 7250 5325 50  0000 C CNN
-F 1 "Jumper" H 7250 5416 50  0000 C CNN
-F 2 "kbd:Jumper" H 7250 5550 50  0001 C CNN
-F 3 "~" H 7250 5550 50  0001 C CNN
-	1    7250 5550
-	-1   0    0    1
 $EndComp
 $Comp
@@
 	1    6400 5600
 	1    0    0    -1
-$EndComp
-$Comp
-L Connector_Generic:Conn_01x01 J1
-U 1 1 5E056F6B
-P 6775 5125
-F 0 "J1" V 6739 5037 50  0000 R CNN
-F 1 "i2c-pin" V 6648 5037 50  0000 R CNN
-F 2 "kbd:1pin_conn" H 6775 5125 50  0001 C CNN
-F 3 "~" H 6775 5125 50  0001 C CNN
-	1    6775 5125
-	0    -1   -1   0
-$EndComp
-$Comp
-L Connector_Generic:Conn_01x01 J3
-U 1 1 5E057B6E
-P 6775 5925
-F 0 "J3" V 6647 6005 50  0000 L CNN
-F 1 "i2c-pin" V 6738 6005 50  0000 L CNN
-F 2 "kbd:1pin_conn" H 6775 5925 50  0001 C CNN
-F 3 "~" H 6775 5925 50  0001 C CNN
-	1    6775 5925
-	0    1    1    0
 $EndComp
 $Comp
@@
 Wire Wire Line
 	6400 5500 6075 5500
-Wire Wire Line
-	6075 5400 6775 5400
-Wire Wire Line
-	6775 5400 6775 5325
-Wire Wire Line
-	6075 5550 6775 5550
-Wire Wire Line
-	6775 5550 6775 5725
-Wire Wire Line
-	6950 5550 6775 5550
-Connection ~ 6775 5550
-Text GLabel 7550 5550 2    50   Input ~ 0
+Text GLabel 6950 5550 2    50   Input ~ 0
 data
 Text GLabel 4350 6450 2    50   Input ~ 0
@@
 F 0 "SW27" H 7600 4480 50  0000 C CNN
 F 1 "SW_PUSH" H 7600 4389 50  0000 C CNN
-F 2 "MX_Alps_Hybrid:MX-1U-NoLED" H 7600 4225 50  0001 C CNN
+F 2 "MX_Alps_Hybrid:MX-1.5U-NoLED" H 7600 4225 50  0001 C CNN
 F 3 "" H 7600 4225 50  0000 C CNN
 	1    7600 4225
@@
 NoConn ~ 1275 5750
 NoConn ~ 1275 5850
-NoConn ~ 4550 -975
+NoConn ~ 6075 5400
+Wire Wire Line
+	6075 5550 6950 5550
 $EndSCHEMATC
