File: iroha60/pcb/iroha60-left/iroha60-left.kicad_pcb (KiCad board)
At the start: 2 copper layers, 63 parts, among them J1 i2c-pin, J2 MJ-4PP-9, J3 i2c-pin, J4 LED, SW1 SW_PUSH, SW10 SW_PUSH, SW11 SW_PUSH, SW12 SW_PUSH, SW13 SW_PUSH, SW14 SW_PUSH, SW15 SW_PUSH, SW16 SW_PUSH, SW17 SW_PUSH, SW18 SW_PUSH, SW19 SW_PUSH, SW2 SW_PUSH, SW20 SW_PUSH, SW21 SW_PUSH, SW22 SW_PUSH, SW23 SW_PUSH, SW24 SW_PUSH, SW25 SW_PUSH, SW26 SW_PUSH, SW27 SW_PUSH, SW28 SW_PUSH, SW29 RESET_SW, SW3 SW_PUSH, SW4 SW_PUSH, SW5 SW_PUSH, SW6 SW_PUSH, SW7 SW_PUSH, SW8 SW_PUSH, SW9 SW_PUSH, U1 ProMicro

Commit message: Updated
Parts:
- U1: footprint kbd:ProMicro_v3.5 -> kbd:ProMicro_v3
- moved D14 94.4 mm to (66.4, 207.7)
- moved D24 94.4 mm to (56.4, 207.7)
- moved D25 94.4 mm to (46.4, 207.7)
- moved D9 94.4 mm to (76.4, 207.7)
- moved SW25 94.4 mm to (81.2, 188.3)
- moved SW27 94.4 mm to (56.3, 188.3)
- moved D11 94.4 mm to (76.4, 202.4)
- moved D13 94.4 mm to (66.4, 210.3)
- moved D18 94.4 mm to (66.4, 202.4)
- moved D19 94.4 mm to (56.4, 210.3)
- moved D2 94.4 mm to (46.4, 202.4)
- moved D21 94.4 mm to (46.4, 215.6)
- moved D23 94.4 mm to (46.4, 210.3)
- moved D28 94.4 mm to (56.4, 202.4)
- moved D3 94.4 mm to (56.4, 215.6)
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
Commit message: Updated
Parts:
- SW27: footprint MX_Alps_Hybrid:MX-1.5U-NoLED -> MX_Alps_Hybrid:MX-1U-NoLED
- U1: footprint kbd:ProMicro_v3 -> kbd:ProMicro_v2_1side
- moved SW21 161.9 mm to (35.0, 223.8)
- moved D7 159.5 mm to (205.9, 135.6)
- moved D8 150.8 mm to (205.9, 132.9)
- moved SW29 126.7 mm to (205.6, 139.2)
- moved SW24 118.7 mm to (53.9, 203.6)
- moved SW12 118.7 mm to (75.4, 223.8)
- moved D10 117.6 mm to (184.4, 158.4)
- moved D11 117.6 mm to (184.4, 155.8)
- moved D12 117.6 mm to (184.4, 153.1)
- moved D5 111.9 mm to (170.0, 173.3)
- moved J2 108.4 mm to (197.3, 132.3)
- moved SW1 93.6 mm to (115.8, 222.5)
- moved SW19 90.3 mm to (55.2, 223.8)
- moved U1 88.5 mm to (34.3, 192.1)
- moved D6 75.9 mm to (149.8, 193.5)
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
Commit message: Updated
Parts:
- removed J1, J3: i2c-pin, kbd:1pin_conn
- removed JP1: Jumper, kbd:Jumper
- added REF**: MountingHole_2.2mm_M2, MountingHole:MountingHole_2.2mm_M2, F.Cu at (146.3, 75.6)
- added REF**: MountingHole_2.2mm_M2, MountingHole:MountingHole_2.2mm_M2, F.Cu at (21.7, 75.6)
- added REF**: MountingHole_2.2mm_M2, MountingHole:MountingHole_2.2mm_M2, F.Cu at (138.7, 111.6)
- added REF**: MountingHole_2.2mm_M2, MountingHole:MountingHole_2.2mm_M2, F.Cu at (67.3, 111.7)
- added REF**: MountingHole_2.2mm_M2, MountingHole:MountingHole_2.2mm_M2, F.Cu at (91.1, 56.5)
- added REF**: MountingHole_2.2mm_M2, MountingHole:MountingHole_2.2mm_M2, F.Cu at (134.0, 20.4)
- added REF**: MountingHole_2.2mm_M2, MountingHole:MountingHole_2.2mm_M2, F.Cu at (38.7, 20.4)
- J2, J4, SW29, U1: moved to B.Cu
- SW27: footprint MX_Alps_Hybrid:MX-1U-NoLED -> MX_Alps_Hybrid:MX-1.5U-NoLED
- moved SW1 212.9 mm to (29.2, 27.9)
- moved D3 212.4 mm to (75.3, 27.9), turned to 90 degrees
- moved D2 208.9 mm to (56.2, 27.9), turned to 90 degrees
- moved D4 206.6 mm to (94.4, 27.9), turned to 90 degrees
- moved SW29 197.6 mm to (22.1, 66.0), turned to 90 degrees
- moved SW6 197.3 mm to (124.5, 27.9)
- moved D9 195.4 mm to (68.8, 46.9), turned to 90 degrees
- moved D13 189.3 mm to (126.0, 47.0), turned to 90 degrees
- moved SW2 187.5 mm to (48.3, 27.9)
- moved SW3 186.9 mm to (67.3, 27.9)
- moved SW12 181.1 mm to (114.9, 47.0)
- moved D1 181.0 mm to (37.2, 27.9), turned to 90 degrees
- moved D14 180.2 mm to (44.4, 65.8), turned to 90 degrees
- moved SW19 178.5 mm to (138.7, 66.0)
- moved D18 178.3 mm to (127.7, 66.0), turned to 90 degrees
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Connections:
- J2 pad B: Net-(J2-PadB) -> data
Other:
- board outline added: 138.1 x 95.2 mm

Commit message: Updated
Routing:
- net GND: track 0.00 -> 312.6 mm, vias 0 -> 2
- net col6: track 0.00 -> 221.8 mm, vias 0 -> 1
- net VCC: track 0.00 -> 218.2 mm, vias 0 -> 4
- net col5: track 0.00 -> 192.4 mm, vias 0 -> 9
- net col4: track 0.00 -> 180.5 mm, vias 0 -> 8
- net row3: track 0.00 -> 154.3 mm, vias 0 -> 1
- net row0: track 0.00 -> 150.6 mm
- net row4: track 0.00 -> 137.5 mm, vias 0 -> 1
- net row2: track 0.00 -> 130.4 mm, vias 0 -> 1
- net led: track 0.00 -> 129.9 mm, vias 0 -> 3
- net data: track 0.00 -> 116.1 mm, vias 0 -> 5
- net row1: track 0.00 -> 110.8 mm
- net col3: track 0.00 -> 98.8 mm, vias 0 -> 6
- net col2: track 0.00 -> 84.3 mm, vias 0 -> 5
- net col1: track 0.00 -> 65.3 mm, vias 0 -> 2
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- added copper zone on B.Cu, net (none)
- added copper zone on F.Cu, net (none)

Commit message: Updated
Parts:
- moved J4 81.7 mm to (57.1, 77.6)
Routing:
- net GND: track 312.6 -> 193.9 mm, vias 2 -> 4
- net led: track 129.9 -> 47.6 mm
- net VCC: track 218.2 -> 144.4 mm
Changed lines of the file:
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@@
     (thickness 1.6)
     (drawings 12)
-    (tracks 530)
+    (tracks 529)
     (zones 0)
     (modules 67)
@@
   )
   (setup
-    (last_trace_width 0.5)
+    (last_trace_width 0.25)
     (user_trace_width 0.5)
     (trace_clearance 0.2)
@@
   )
   (module kbd:StripLED_1side (layer B.Cu)
-    (at 138.785 77.53)
+    (at 57.07875 77.58)
     (fp_text reference J4 (at 0 2.54) (layer B.SilkS) hide
       (effects (font (size 1 1) (thickness 0.15)) (justify mirror))
@@
       (effects (font (size 1 1) (thickness 0.15)) (justify mirror))
     )
-    (fp_text user VCC (at -2.75 -0.1) (layer B.SilkS)
+    (fp_text user VCC (at 2.75 -5) (layer B.SilkS)
       (effects (font (size 1 1) (thickness 0.15)) (justify mirror))
     )
-    (fp_text user LED (at -2.71 -2.56) (layer B.SilkS)
+    (fp_text user LED (at 2.75 -2.56) (layer B.SilkS)
       (effects (font (size 1 1) (thickness 0.15)) (justify mirror))
     )
-    (fp_text user GND (at -2.8 -5.15) (layer B.SilkS)
+    (fp_text user GND (at 2.75 0) (layer B.SilkS)
       (effects (font (size 1 1) (thickness 0.15)) (justify mirror))
     )
@@
   (segment (start 31.685 51.015) (end 31.685 51.5359) (width 0.5) (layer B.Cu) (net 34))
   (segment (start 46.516862 53.015) (end 45.185 53.015) (width 0.5) (layer B.Cu) (net 34))
-  (segment (start 47.566501 89.538501) (end 47.566501 54.064639) (width 0.5) (layer B.Cu) (net 34))
-  (segment (start 57.234999 100.023001) (end 57.234999 99.206999) (width 0.5) (layer B.Cu) (net 34))
-  (segment (start 59.026998 101.815) (end 57.234999 100.023001) (width 0.5) (layer B.Cu) (net 34))
-  (segment (start 62.485 101.815) (end 59.026998 101.815) (width 0.5) (layer B.Cu) (net 34))
-  (segment (start 69.9 77.53) (end 59.568999 87.861001) (width 0.5) (layer B.Cu) (net 34))
-  (segment (start 59.568999 95.098999) (end 62.485 98.015) (width 0.5) (layer B.Cu) (net 34))
-  (segment (start 57.234999 99.206999) (end 47.566501 89.538501) (width 0.5) (layer B.Cu) (net 34))
-  (segment (start 59.568999 87.861001) (end 59.568999 95.098999) (width 0.5) (layer B.Cu) (net 34))
-  (segment (start 62.485 98.015) (end 62.485 101.815) (width 0.5) (layer B.Cu) (net 34))
   (segment (start 47.566501 54.064639) (end 46.516862 53.015) (width 0.5) (layer B.Cu) (net 34))
-  (segment (start 138.785 77.53) (end 69.9 77.53) (width 0.5) (layer B.Cu) (net 34))
   (segment (start 32.285 33.1759) (end 26.796499 38.664401) (width 0.5) (layer B.Cu) (net 34))
   (segment (start 32.285 26.715) (end 32.285 33.1759) (width 0.5) (layer B.Cu) (net 34))
@@
   (segment (start 26.796499 38.664401) (end 26.0345 39.4264) (width 0.5) (layer B.Cu) (net 34))
   (segment (start 112.835 24.715) (end 112.835 24.315) (width 0.5) (layer B.Cu) (net 34))
+  (via (at 49.07875 78.58) (size 0.8) (drill 0.4) (layers F.Cu B.Cu) (net 34))
+  (segment (start 47.566501 77.067751) (end 49.07875 78.58) (width 0.5) (layer B.Cu) (net 34))
+  (segment (start 47.566501 54.064639) (end 47.566501 77.067751) (width 0.5) (layer B.Cu) (net 34))
+  (via (at 51.82875 80.58) (size 0.8) (drill 0.4) (layers F.Cu B.Cu) (net 34))
+  (segment (start 49.82875 78.58) (end 51.82875 80.58) (width 0.5) (layer F.Cu) (net 34))
+  (segment (start 49.07875 78.58) (end 49.82875 78.58) (width 0.5) (layer F.Cu) (net 34))
+  (segment (start 57.07875 78.842) (end 57.07875 77.58) (width 0.5) (layer B.Cu) (net 34))
+  (segment (start 55.34075 80.58) (end 57.07875 78.842) (width 0.5) (layer B.Cu) (net 34))
+  (segment (start 51.82875 80.58) (end 55.34075 80.58) (width 0.5) (layer B.Cu) (net 34))
   (via (at 38.485 35.715) (size 0.8) (drill 0.4) (layers F.Cu B.Cu) (net 35))
   (segment (start 39.058002 35.715) (end 38.485 35.715) (width 0.25) (layer B.Cu) (net 35))
@@
   (segment (start 32.485 36.715) (end 31.1145 38.0855) (width 0.25) (layer B.Cu) (net 35))
   (via (at 48.785 52.115) (size 0.8) (drill 0.4) (layers F.Cu B.Cu) (net 35))
-  (segment (start 70.228328 72.45) (end 64.991401 67.213073) (width 0.5) (layer B.Cu) (net 35))
-  (segment (start 52.453502 52.115) (end 48.785 52.115) (width 0.5) (layer B.Cu) (net 35))
-  (segment (start 64.991401 64.652899) (end 52.453502 52.115) (width 0.5) (layer B.Cu) (net 35))
-  (segment (start 64.991401 67.213073) (end 64.991401 64.652899) (width 0.5) (layer B.Cu) (net 35))
-  (segment (start 138.785 72.45) (end 70.228328 72.45) (width 0.5) (layer B.Cu) (net 35))
   (via (at 34.185 43.515) (size 0.8) (drill 0.4) (layers F.Cu B.Cu) (net 35))
   (segment (start 34.185 42.4969) (end 31.1145 39.4264) (width 0.5) (layer B.Cu) (net 35))
@@
   (segment (start 35.480526 52.115) (end 31.185 47.819474) (width 0.5) (layer F.Cu) (net 35))
   (segment (start 48.785 52.115) (end 35.480526 52.115) (width 0.5) (layer F.Cu) (net 35))
+  (segment (start 55.81675 72.5) (end 57.07875 72.5) (width 0.5) (layer B.Cu) (net 35))
+  (segment (start 52.646501 69.329751) (end 55.81675 72.5) (width 0.5) (layer B.Cu) (net 35))
+  (segment (start 52.646501 53.397751) (end 52.646501 69.329751) (width 0.5) (layer B.Cu) (net 35))
+  (segment (start 51.36375 52.115) (end 52.646501 53.397751) (width 0.5) (layer B.Cu) (net 35))
+  (segment (start 48.785 52.115) (end 51.36375 52.115) (width 0.5) (layer B.Cu) (net 35))
   (via (at 26.085 62.815) (size 0.8) (drill 0.4) (layers F.Cu B.Cu) (net 36))
   (segment (start 23.4945 60.2245) (end 26.085 62.815) (width 0.25) (layer F.Cu) (net 36))
@@
   (segment (start 39.685 76.415) (end 45.085 76.415) (width 0.25) (layer B.Cu) (net 36))
   (segment (start 26.085 62.815) (end 39.685 76.415) (width 0.25) (layer B.Cu) (net 36))
-  (via (at 59.685 72.915) (size 0.8) (drill 0.4) (layers F.Cu B.Cu) (net 36))
-  (segment (start 58.083901 74.516099) (end 59.685 72.915) (width 0.25) (layer F.Cu) (net 36))
-  (segment (start 46.983901 74.516099) (end 58.083901 74.516099) (width 0.25) (layer F.Cu) (net 36))
   (segment (start 45.085 76.415) (end 46.983901 74.516099) (width 0.25) (layer F.Cu) (net 36))
-  (segment (start 61.76 74.99) (end 138.785 74.99) (width 0.25) (layer B.Cu) (net 36))
-  (segment (start 59.685 72.915) (end 61.76 74.99) (width 0.25) (layer B.Cu) (net 36))
+  (segment (start 53.642651 74.516099) (end 54.57875 73.58) (width 0.25) (layer F.Cu) (net 36))
+  (via (at 54.57875 73.58) (size 0.8) (drill 0.4) (layers F.Cu B.Cu) (net 36))
+  (segment (start 46.983901 74.516099) (end 53.642651 74.516099) (width 0.25) (layer F.Cu) (net 36))
+  (segment (start 56.03875 75.04) (end 57.07875 75.04) (width 0.25) (layer B.Cu) (net 36))
+  (segment (start 54.57875 73.58) (end 56.03875 75.04) (width 0.25) (layer B.Cu) (net 36))
   (via (at 42.085 20.215) (size 0.8) (drill 0.4) (layers F.Cu B.Cu) (net 37))
   (segment (start 110.235 20.215) (end 42.085 20.215) (width 0.25) (layer B.Cu) (net 37))

Commit message: Updated
Other:
- board text added: "iroha60 rev.1 Designed by kironono"
Changed lines of the file:
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@@
   (general
     (thickness 1.6)
-    (drawings 12)
+    (drawings 13)
     (tracks 529)
     (zones 0)
@@
     (pad "" np_thru_hole circle (at 5.08 0 48.0996) (size 1.75 1.75) (drill 1.75) (layers *.Cu *.Mask))
   )
+  (gr_text "iroha60 rev.1\nDesigned by kironono" (at 81.07875 110.83) (layer F.SilkS)
+    (effects (font (size 1.5 1.5) (thickness 0.3)))
+  )
   (gr_line (start 19.685 113.665) (end 19.685 18.415) (layer Edge.Cuts) (width 0.05))
