File: iroha60/pcb/iroha60-left/iroha60-left.kicad_pcb (KiCad board)
At the start: 2 copper layers, 138.1 x 95.2 mm, 67 parts, among them J2 MJ-4PP-9, J4 LED, SW1 SW_PUSH, SW10 SW_PUSH, SW11 SW_PUSH, SW12 SW_PUSH, SW13 SW_PUSH, SW14 SW_PUSH, SW15 SW_PUSH, SW16 SW_PUSH, SW17 SW_PUSH, SW18 SW_PUSH, SW19 SW_PUSH, SW2 SW_PUSH, SW20 SW_PUSH, SW21 SW_PUSH, SW22 SW_PUSH, SW23 SW_PUSH, SW24 SW_PUSH, SW25 SW_PUSH, SW26 SW_PUSH, SW27 SW_PUSH, SW28 SW_PUSH, SW29 RESET_SW, SW3 SW_PUSH, SW4 SW_PUSH, SW5 SW_PUSH, SW6 SW_PUSH, SW7 SW_PUSH, SW8 SW_PUSH, SW9 SW_PUSH, U1 ProMicro

Commit message: Updated
Parts:
- moved D28 32.5 mm to (97.6, 104.1)
- moved D20 12.0 mm to (61.1, 85.1)
- moved D26 0.19 mm to (65.8, 104.1)
- moved D27 0.19 mm to (89.6, 104.1)
Routing:
- net row4: track 137.5 -> 105.0 mm
- net Net-(D28-Pad2): track 9.93 -> 42.0 mm
- net Net-(D20-Pad2): track 10.1 -> 22.6 mm
Changed lines of the file:
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@@
     (thickness 1.6)
     (drawings 15)
-    (tracks 529)
+    (tracks 538)
     (zones 0)
     (modules 67)
@@
     (solder_mask_min_width 0.25)
     (aux_axis_origin 0 0)
-    (grid_origin 19.685 18.415)
+    (grid_origin 72.0725 85.09)
     (visible_elements FFFFFF7F)
     (pcbplotparams
@@
     (tags "mounting hole 2.2mm no annular m2")
     (attr virtual)
-    (fp_text reference REF** (at 0 -3.2) (layer F.SilkS)
+    (fp_text reference REF** (at 0 -3.2) (layer Dwgs.User)
       (effects (font (size 1 1) (thickness 0.15)))
     )
@@
   )
   (module kbd:D3_TH_SMD (layer F.Cu)
-    (at 49.11625 85.09 90)
+    (at 61.0725 85.09 90)
     (descr "Resitance 3 pas")
     (tags R)
@@
   )
   (module kbd:D3_TH_SMD (layer F.Cu)
-    (at 65.785 104.33 90)
+    (at 65.785 104.14 90)
     (descr "Resitance 3 pas")
     (tags R)
@@
   )
   (module kbd:D3_TH_SMD (layer F.Cu)
-    (at 89.5975 104.33 90)
+    (at 89.5975 104.14 90)
     (descr "Resitance 3 pas")
     (tags R)
@@
   )
   (module kbd:D3_TH_SMD (layer F.Cu)
-    (at 130.07875 104.33 90)
+    (at 97.5975 104.14 90)
     (descr "Resitance 3 pas")
     (tags R)
@@
   (segment (start 130.7475 62.13) (end 133.042499 59.835001) (width 0.25) (layer F.Cu) (net 22))
   (segment (start 130.7475 64.165) (end 130.7475 62.13) (width 0.25) (layer B.Cu) (net 22))
-  (segment (start 49.11625 83.315) (end 49.11625 81.28) (width 0.25) (layer F.Cu) (net 23))
   (segment (start 44.92625 81.28) (end 43.65625 80.01) (width 0.25) (layer F.Cu) (net 23))
   (segment (start 49.11625 81.28) (end 44.92625 81.28) (width 0.25) (layer F.Cu) (net 23))
-  (segment (start 49.11625 83.315) (end 49.11625 81.28) (width 0.25) (layer B.Cu) (net 23))
+  (segment (start 60.374001 81.978499) (end 61.0725 81.28) (width 0.25) (layer F.Cu) (net 23))
+  (segment (start 49.814749 81.978499) (end 60.374001 81.978499) (width 0.25) (layer F.Cu) (net 23))
+  (segment (start 49.11625 81.28) (end 49.814749 81.978499) (width 0.25) (layer F.Cu) (net 23))
+  (segment (start 61.0725 81.28) (end 61.0725 83.315) (width 0.25) (layer F.Cu) (net 23))
+  (segment (start 61.0725 83.315) (end 61.0725 81.28) (width 0.25) (layer B.Cu) (net 23))
   (segment (start 140.2725 89.09) (end 140.2725 87.055) (width 0.25) (layer F.Cu) (net 24))
   (segment (start 139.324 89.09) (end 137.2225 89.09) (width 0.25) (layer F.Cu) (net 24))
@@
   (segment (start 98.9325 88.9) (end 99.1225 89.09) (width 0.25) (layer F.Cu) (net 24))
   (segment (start 80.0725 88.9) (end 98.9325 88.9) (width 0.25) (layer F.Cu) (net 24))
-  (segment (start 49.11625 86.865) (end 49.11625 88.9) (width 0.25) (layer F.Cu) (net 24))
-  (segment (start 49.11625 88.9) (end 80.0725 88.9) (width 0.25) (layer F.Cu) (net 24))
-  (segment (start 49.11625 86.865) (end 49.11625 88.9) (width 0.25) (layer B.Cu) (net 24))
   (segment (start 80.0725 86.865) (end 80.0725 88.9) (width 0.25) (layer B.Cu) (net 24))
   (segment (start 99.1225 87.055) (end 99.1225 89.09) (width 0.25) (layer B.Cu) (net 24))
@@
   (segment (start 46.37 88.9) (end 49.11625 88.9) (width 0.25) (layer F.Cu) (net 24))
   (segment (start 44.385001 86.915001) (end 46.37 88.9) (width 0.25) (layer F.Cu) (net 24))
+  (segment (start 49.11625 88.9) (end 61.0725 88.9) (width 0.25) (layer F.Cu) (net 24))
+  (segment (start 61.0725 86.865) (end 61.0725 88.9) (width 0.25) (layer F.Cu) (net 24))
+  (segment (start 61.0725 88.9) (end 80.0725 88.9) (width 0.25) (layer F.Cu) (net 24))
+  (segment (start 61.0725 86.865) (end 61.0725 88.9) (width 0.25) (layer B.Cu) (net 24))
   (segment (start 80.0725 83.315) (end 80.0725 81.28) (width 0.25) (layer F.Cu) (net 25))
   (segment (start 75.8825 81.28) (end 74.6125 80.01) (width 0.25) (layer F.Cu) (net 25))
@@
   (segment (start 142.3675 81.47) (end 144.952499 78.885001) (width 0.25) (layer F.Cu) (net 29))
   (segment (start 140.2725 83.505) (end 140.2725 81.47) (width 0.25) (layer B.Cu) (net 29))
-  (segment (start 130.07875 108.14) (end 130.07875 106.105) (width 0.25) (layer F.Cu) (net 30))
-  (segment (start 89.5975 106.105) (end 89.5975 108.14) (width 0.25) (layer F.Cu) (net 30))
-  (segment (start 65.785 106.105) (end 65.785 108.14) (width 0.25) (layer F.Cu) (net 30))
-  (segment (start 110.389228 108.14) (end 89.5975 108.14) (width 0.25) (layer F.Cu) (net 30))
-  (segment (start 130.07875 108.14) (end 110.389228 108.14) (width 0.25) (layer F.Cu) (net 30))
-  (segment (start 89.5975 108.14) (end 65.785 108.14) (width 0.25) (layer F.Cu) (net 30))
-  (segment (start 130.07875 106.105) (end 130.07875 108.14) (width 0.25) (layer B.Cu) (net 30))
-  (segment (start 89.5975 106.105) (end 89.5975 108.14) (width 0.25) (layer B.Cu) (net 30))
-  (segment (start 65.785 106.105) (end 65.785 108.14) (width 0.25) (layer B.Cu) (net 30))
   (segment (start 58.085 94.369228) (end 58.085 99.615) (width 0.25) (layer B.Cu) (net 30))
   (segment (start 50.139751 86.423979) (end 58.085 94.369228) (width 0.25) (layer B.Cu) (net 30))
@@
   (via (at 58.085 99.615) (size 0.8) (drill 0.4) (layers F.Cu B.Cu) (net 30))
   (segment (start 48.8945 54.6464) (end 50.139751 55.891651) (width 0.25) (layer B.Cu) (net 30))
-  (segment (start 64.8365 108.14) (end 65.785 108.14) (width 0.25) (layer F.Cu) (net 30))
-  (segment (start 60.103901 103.407401) (end 64.8365 108.14) (width 0.25) (layer F.Cu) (net 30))
   (segment (start 60.103901 101.633901) (end 60.103901 103.407401) (width 0.25) (layer F.Cu) (net 30))
   (segment (start 58.085 99.615) (end 60.103901 101.633901) (width 0.25) (layer F.Cu) (net 30))
-  (segment (start 65.785 102.555) (end 65.785 100.52) (width 0.25) (layer F.Cu) (net 31))
-  (segment (start 60.905 99.64) (end 60.285 99.64) (width 0.25) (layer F.Cu) (net 31))
-  (segment (start 61.785 100.52) (end 60.905 99.64) (width 0.25) (layer F.Cu) (net 31))
-  (segment (start 65.785 100.52) (end 61.785 100.52) (width 0.25) (layer F.Cu) (net 31))
-  (segment (start 65.785 102.555) (end 65.785 100.52) (width 0.25) (layer B.Cu) (net 31))
-  (segment (start 89.5975 102.555) (end 89.5975 100.52) (width 0.25) (layer F.Cu) (net 32))
+  (segment (start 97.5975 105.915) (end 97.5975 107.95) (width 0.25) (layer F.Cu) (net 30))
+  (segment (start 97.5975 105.915) (end 97.5975 107.95) (width 0.25) (layer B.Cu) (net 30))
+  (segment (start 64.6465 107.95) (end 65.785 107.95) (width 0.25) (layer F.Cu) (net 30))
+  (segment (start 60.103901 103.407401) (end 64.6465 107.95) (width 0.25) (layer F.Cu) (net 30))
+  (segment (start 65.785 105.915) (end 65.785 107.95) (width 0.25) (layer F.Cu) (net 30))
+  (segment (start 65.785 105.915) (end 65.785 107.95) (width 0.25) (layer B.Cu) (net 30))
+  (segment (start 66.7335 107.95) (end 89.5975 107.95) (width 0.25) (layer F.Cu) (net 30))
+  (segment (start 65.785 107.95) (end 66.7335 107.95) (width 0.25) (layer F.Cu) (net 30))
+  (segment (start 89.5975 105.915) (end 89.5975 107.95) (width 0.25) (layer F.Cu) (net 30))
+  (segment (start 89.5975 105.915) (end 89.5975 107.95) (width 0.25) (layer B.Cu) (net 30))
+  (segment (start 89.5975 107.95) (end 97.5975 107.95) (width 0.25) (layer F.Cu) (net 30))
+  (segment (start 65.785 102.365) (end 65.785 100.33) (width 0.25) (layer F.Cu) (net 31))
+  (segment (start 65.785 100.33) (end 65.785 102.365) (width 0.25) (layer B.Cu) (net 31))
+  (segment (start 62.205 100.94) (end 65.175 100.94) (width 0.25) (layer F.Cu) (net 31))
+  (segment (start 60.905 99.64) (end 62.205 100.94) (width 0.25) (layer F.Cu) (net 31))
+  (segment (start 65.175 100.94) (end 65.785 100.33) (width 0.25) (layer F.Cu) (net 31))
+  (segment (start 60.285 99.64) (end 60.905 99.64) (width 0.25) (layer F.Cu) (net 31))
+  (segment (start 89.5975 102.365) (end 89.5975 100.33) (width 0.25) (layer F.Cu) (net 32))
   (segment (start 84.7175 99.64) (end 84.0975 99.64) (width 0.25) (layer F.Cu) (net 32))
-  (segment (start 85.5975 100.52) (end 84.7175 99.64) (width 0.25) (layer F.Cu) (net 32))
-  (segment (start 89.5975 100.52) (end 85.5975 100.52) (width 0.25) (layer F.Cu) (net 32))
-  (segment (start 89.5975 102.555) (end 89.5975 100.52) (width 0.25) (layer B.Cu) (net 32))
-  (segment (start 130.07875 102.555) (end 130.07875 100.52) (width 0.25) (layer F.Cu) (net 33))
+  (segment (start 85.4075 100.33) (end 84.7175 99.64) (width 0.25) (layer F.Cu) (net 32))
+  (segment (start 89.5975 100.33) (end 85.4075 100.33) (width 0.25) (layer F.Cu) (net 32))
+  (segment (start 89.5975 102.365) (end 89.5975 100.33) (width 0.25) (layer B.Cu) (net 32))
   (segment (start 125.19875 99.64) (end 124.57875 99.64) (width 0.25) (layer F.Cu) (net 33))
-  (segment (start 126.07875 100.52) (end 125.19875 99.64) (width 0.25) (layer F.Cu) (net 33))
-  (segment (start 130.07875 100.52) (end 126.07875 100.52) (width 0.25) (layer F.Cu) (net 33))
-  (segment (start 130.07875 102.555) (end 130.07875 100.52) (width 0.25) (layer B.Cu) (net 33))
+  (segment (start 97.5975 102.365) (end 97.5975 100.33) (width 0.25) (layer F.Cu) (net 33))
+  (segment (start 97.5975 100.33) (end 97.5975 102.365) (width 0.25) (layer B.Cu) (net 33))
+  (segment (start 124.61875 100.65099) (end 124.61875 99.06) (width 0.25) (layer F.Cu) (net 33))
+  (segment (start 124.885 100.91724) (end 124.61875 100.65099) (width 0.25) (layer F.Cu) (net 33))
+  (segment (start 124.885 105.54) (end 124.885 100.91724) (width 0.25) (layer F.Cu) (net 33))
+  (segment (start 123.385 107.04) (end 124.885 105.54) (width 0.25) (layer F.Cu) (net 33))
+  (segment (start 104.3075 107.04) (end 123.385 107.04) (width 0.25) (layer F.Cu) (net 33))
+  (segment (start 97.5975 100.33) (end 104.3075 107.04) (width 0.25) (layer F.Cu) (net 33))
   (segment (start 28.5745 62.78175) (end 22.06625 69.29) (width 0.5) (layer F.Cu) (net 34))
   (segment (start 28.5745 54.6464) (end 28.5745 62.78175) (width 0.5) (layer F.Cu) (net 34))

Commit message: Updated
Parts:
- moved REF** 7.53 mm to (146.3, 111.7)
Changed lines of the file:
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@@
     (solder_mask_min_width 0.25)
     (aux_axis_origin 0 0)
-    (grid_origin 72.0725 85.09)
+    (grid_origin 148.2725 75.565)
     (visible_elements FFFFFF7F)
     (pcbplotparams
@@
       (drillshape 0)
       (scaleselection 1)
-      (outputdirectory "publish_rev1/"))
+      (outputdirectory "iroha60-left-pub-rev1_1/"))
   )
   (net 0 "")
@@
   )
   (module MountingHole:MountingHole_2.2mm_M2 (layer F.Cu)
-    (at 138.7475 111.615)
+    (at 146.2725 111.665)
     (descr "Mounting Hole 2.2mm, no annular, M2")
     (tags "mounting hole 2.2mm no annular m2")

Commit message: Updated
Other:
- board text added: "iroha60 rev.1 2020-08-12 Designed by kironono"
- board text removed: "iroha60 rev.1 Designed by kironono"
Changed lines of the file:
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@@
     (arrow2b (pts (xy 19.685 13.6525) (xy 20.811504 13.066079)))
   )
-  (gr_text "iroha60 rev.1\nDesigned by kironono" (at 81.07875 110.83) (layer F.SilkS)
+  (gr_text "iroha60 rev.1 2020-08-12\nDesigned by kironono" (at 81.07875 110.83) (layer F.SilkS)
     (effects (font (size 1.5 1.5) (thickness 0.3)))
   )
