File: iroha60/pcb/iroha60-right/iroha60-right.kicad_pcb (KiCad board)
At the start: 2 copper layers, 89 parts, among them J1 i2c-pin, J2 MJ-4PP-9, J3 i2c-pin, J4 LED, SW1 SW_PUSH, SW10 SW_PUSH, SW11 SW_PUSH, SW12 SW_PUSH, SW13 SW_PUSH, SW14 SW_PUSH, SW15 SW_PUSH, SW16 SW_PUSH, SW17 SW_PUSH, SW18 SW_PUSH, SW19 SW_PUSH, SW2 SW_PUSH, SW20 SW_PUSH, SW21 SW_PUSH, SW22 SW_PUSH, SW23 SW_PUSH, SW24 SW_PUSH, SW25 SW_PUSH, SW26 SW_PUSH, SW27 SW_PUSH, SW28 SW_PUSH, SW29 SW_PUSH, SW3 SW_PUSH, SW30 SW_PUSH, SW31 SW_PUSH, SW32 SW_PUSH, SW33 SW_PUSH, SW34 SW_PUSH, SW35 SW_PUSH, SW36 SW_PUSH, SW37 SW_PUSH, SW38 SW_PUSH, SW39 SW_PUSH, SW4 SW_PUSH, SW40 SW_PUSH, SW41 SW_PUSH, SW42 RESET_SW, SW5 SW_PUSH, SW6 SW_PUSH, SW7 SW_PUSH, SW8 SW_PUSH, SW9 SW_PUSH, U1 ProMicro

Commit message: Updated
Parts:
- removed D34, D35, D36, D37, D38, D39, D40, D41: D, kbd:D3_TH_SMD
- removed SW35, SW38, SW39, SW40, SW41: SW_PUSH, MX_Alps_Hybrid:MX-1U-NoLED
- removed SW36: SW_PUSH, MX_Alps_Hybrid:MX-2.25U-ReversedStabilizers-NoLED
- removed SW37: SW_PUSH, MX_Alps_Hybrid:MX-1.5U-NoLED
- removed SW42: RESET_SW, kbd:ResetSW_1side
- SW16: footprint MX_Alps_Hybrid:MX-1U-NoLED -> MX_Alps_Hybrid:MX-1.5U-NoLED
- SW17: footprint MX_Alps_Hybrid:MX-1.5U-NoLED -> MX_Alps_Hybrid:MX-1U-NoLED
- SW23, SW31: footprint MX_Alps_Hybrid:MX-1U-NoLED -> MX_Alps_Hybrid:MX-2.25U-ReversedStabilizers-NoLED
- SW25: footprint MX_Alps_Hybrid:MX-2.25U-ReversedStabilizers-NoLED -> MX_Alps_Hybrid:MX-1U-NoLED
- SW29: footprint MX_Alps_Hybrid:MX-1U-NoLED -> MX_Alps_Hybrid:MX-1.75U-NoLED
- SW32: footprint MX_Alps_Hybrid:MX-1.75U-NoLED -> MX_Alps_Hybrid:MX-1.5U-NoLED
- SW34: value SW_PUSH -> RESET_SW; footprint MX_Alps_Hybrid:MX-1U-NoLED -> kbd:ResetSW_1side
- U1: footprint kbd:ProMicro_v3.5 -> kbd:ProMicro_v3
- moved D22 197.0 mm to (198.3, 214.5)
- moved D23 179.1 mm to (198.3, 211.9)
- moved D24 179.1 mm to (198.3, 209.2)
- moved D26 177.5 mm to (198.3, 206.6)
- moved J3 170.0 mm to (207.4, 206.8)
- moved D19 167.9 mm to (198.3, 217.2)
- moved D3 161.6 mm to (198.3, 219.8)
- moved J4 146.4 mm to (204.6, 206.5)
- moved D17 141.1 mm to (198.3, 222.5)
- moved SW27 139.9 mm to (29.9, 297.4)
- moved D10 125.2 mm to (190.0, 247.0)
- moved D9 125.2 mm to (190.0, 249.6)
- moved D8 109.1 mm to (190.0, 252.3)
- moved SW34 95.4 mm to (155.8, 288.4)
- moved D5 92.4 mm to (175.7, 267.2)
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Connections:
- D17 pad 1: row1 -> row2
- D18 pad 1: row1 -> row2
- D24 pad 1: row2 -> row3
- D25 pad 1: row2 -> row3
- D26 pad 1: row2 -> row3
- D30 pad 1: row3 -> row4
- D31 pad 1: row3 -> row4
- D32 pad 1: row3 -> row4
- D33 pad 1: row3 -> row4
- D9 pad 1: row0 -> row1
- SW10 pad 1: col0 -> col1
- SW11 pad 1: col1 -> col2
- SW12 pad 1: col2 -> col3
- SW13 pad 1: col3 -> col4
- SW14 pad 1: col4 -> col5
- SW15 pad 1: col5 -> col6
- SW16 pad 1: col6 -> col7
- SW17 pad 1: col7 -> col1
- SW18 pad 1: col8 -> col2
- SW19 pad 1: col1 -> col3
- SW20 pad 1: col2 -> col4
- SW21 pad 1: col3 -> col5
- SW22 pad 1: col4 -> col6
- SW23 pad 1: col5 -> col7
- SW24 pad 1: col6 -> col1
- SW25 pad 1: col7 -> col2
- SW26 pad 1: col8 -> col3
- SW27 pad 1: col1 -> col4
- SW28 pad 1: col2 -> col5
- SW29 pad 1: col3 -> col6
- SW30 pad 1: col4 -> col1
- SW31 pad 1: col5 -> col2
- SW32 pad 1: col6 -> col3
- SW33 pad 1: col7 -> col4
- SW34 pad 1: col8 -> reset
- SW34 pad 2: Net-(D34-Pad2) -> GND
- SW9 pad 1: col8 -> col0
- U1 pad 12: col8 -> Net-(U1-Pad12)

Commit message: Updated
Parts:
- removed J3: i2c-pin, kbd:1pin_conn
- removed J4: LED, kbd:StripLED_1side
- removed JP1: Jumper, kbd:Jumper
- added REF**: MountingHole_2.2mm_M2, MountingHole:MountingHole_2.2mm_M2, F.Cu at (159.9, 81.0)
- added REF**: MountingHole_2.2mm_M2, MountingHole:MountingHole_2.2mm_M2, F.Cu at (35.3, 81.0)
- added REF**: MountingHole_2.2mm_M2, MountingHole:MountingHole_2.2mm_M2, F.Cu at (95.2, 61.9)
- added REF**: MountingHole_2.2mm_M2, MountingHole:MountingHole_2.2mm_M2, F.Cu at (42.9, 117.1)
- added REF**: MountingHole_2.2mm_M2, MountingHole:MountingHole_2.2mm_M2, F.Cu at (114.3, 117.1)
- added REF**: MountingHole_2.2mm_M2, MountingHole:MountingHole_2.2mm_M2, F.Cu at (161.9, 25.8)
- added REF**: MountingHole_2.2mm_M2, MountingHole:MountingHole_2.2mm_M2, F.Cu at (47.6, 25.8)
- J1: value i2c-pin -> MJ-4PP-9; footprint kbd:1pin_conn -> kbd:MJ-4PP-9_1side; moved to B.Cu
- J2: value MJ-4PP-9 -> LED; footprint kbd:MJ-4PP-9_1side -> kbd:StripLED_1side; moved to B.Cu
- SW34: moved to B.Cu
- U1: footprint kbd:ProMicro_v3 -> kbd:ProMicro_v2_1side; moved to B.Cu
- moved D2 275.9 mm to (49.1, 33.3), turned to 90 degrees
- moved SW1 271.8 mm to (38.1, 33.3)
- moved SW8 269.7 mm to (171.4, 33.3)
- moved SW4 265.2 mm to (95.2, 33.3)
- moved D6 262.0 mm to (141.3, 33.3), turned to 90 degrees
- moved SW16 260.7 mm to (166.7, 52.4)
- moved D7 259.7 mm to (160.4, 33.3), turned to 90 degrees
- moved D12 259.7 mm to (93.7, 52.4), turned to 90 degrees
- moved D15 258.4 mm to (131.8, 52.4), turned to 90 degrees
- moved D16 255.9 mm to (134.8, 52.4), turned to 90 degrees
- moved D13 255.5 mm to (112.8, 52.4), turned to 90 degrees
- moved D9 249.9 mm to (36.6, 52.3), turned to 90 degrees
- moved D11 248.1 mm to (74.7, 52.4), turned to 90 degrees
- moved SW2 244.8 mm to (57.1, 33.3)
- moved SW13 244.2 mm to (104.8, 52.4)
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Routing:
- net GND: track 0.00 -> 348.2 mm, vias 0 -> 1
- net VCC: track 0.00 -> 253.4 mm, vias 0 -> 2
- net col1: track 0.00 -> 227.4 mm, vias 0 -> 2
- net col2: track 0.00 -> 196.0 mm, vias 0 -> 8
- net row2: track 0.00 -> 192.8 mm, vias 0 -> 2
- net row3: track 0.00 -> 190.0 mm, vias 0 -> 4
- net col3: track 0.00 -> 183.6 mm, vias 0 -> 8
- net row4: track 0.00 -> 181.3 mm, vias 0 -> 6
- net col4: track 0.00 -> 168.2 mm, vias 0 -> 8
- net col0: track 0.00 -> 167.1 mm, vias 0 -> 1
- net row1: track 0.00 -> 165.5 mm, vias 0 -> 4
- net led: track 0.00 -> 159.3 mm
- net row0: track 0.00 -> 158.3 mm
- net data: track 0.00 -> 122.8 mm
- net col5: track 0.00 -> 114.7 mm, vias 0 -> 6
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- added copper zone on B.Cu, net (none)
- added copper zone on F.Cu, net (none)
Other:
- board outline added: 161.9 x 95.2 mm

Commit message: Updated
Parts:
- added G***: LOGO, logos:logo, F.Cu at (157.8, 125.0)
Other:
- board text added: "iroha60 rev.1 Designed by kironono"

Commit message: Updated
Parts:
- added D34: D, kbd:D3_TH_SMD, F.Cu at (163.4, 90.5)
- added SW35: SW_PUSH, MX_Alps_Hybrid:MX-1U-NoLED, F.Cu at (171.4, 90.5)
- moved REF** 19.0 mm to (179.0, 81.0)
Routing:
- net col7: track 47.8 -> 77.6 mm, vias 1 -> 4
- net Net-(D34-Pad2): track 0.00 -> 16.1 mm
- net row3: track 190.0 -> 203.3 mm
- net row1: track 165.5 -> 168.5 mm
Changed lines of the file:
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@@
     (thickness 1.6)
     (drawings 13)
-    (tracks 679)
+    (tracks 700)
     (zones 0)
-    (modules 78)
-    (nets 57)
+    (modules 80)
+    (nets 58)
   )
   (page A4)
@@
     (solder_mask_min_width 0.25)
     (aux_axis_origin 0 0)
-    (grid_origin 115.825 109.5375)
+    (grid_origin 163.45 90.4875)
     (visible_elements FFFFFF7F)
     (pcbplotparams
@@
   (net 55 "Net-(U1-Pad12)")
   (net 56 "Net-(J1-PadA)")
+  (net 57 "Net-(D34-Pad2)")
   (net_class Default "これはデフォルトのネット クラスです。"
     (clearance 0.2)
@@
     (add_net "Net-(D32-Pad2)")
     (add_net "Net-(D33-Pad2)")
+    (add_net "Net-(D34-Pad2)")
     (add_net "Net-(D4-Pad2)")
     (add_net "Net-(D5-Pad2)")
@@
   )
   (module MountingHole:MountingHole_2.2mm_M2 (layer F.Cu)
-    (at 159.925 80.9625)
+    (at 178.975 80.9625)
     (descr "Mounting Hole 2.2mm, no annular, M2")
     (tags "mounting hole 2.2mm no annular m2")
@@
       (net 41 led))
   )
+  (module kbd:D3_TH_SMD (layer F.Cu)
+    (at 163.45 90.4875 90)
+    (descr "Resitance 3 pas")
+    (tags R)
+    (autoplace_cost180 10)
+    (fp_text reference D34 (at 0 -1.3 90) (layer B.SilkS)
+      (effects (font (size 0.5 0.5) (thickness 0.125)) (justify mirror))
+    )
+    (fp_text value D (at -0.55 0 90) (layer F.Fab) hide
+      (effects (font (size 0.5 0.5) (thickness 0.125)))
+    )
+    (fp_line (start -0.4 0) (end 0.5 -0.5) (layer B.SilkS) (width 0.15))
+    (fp_line (start 0.5 -0.5) (end 0.5 0.5) (layer B.SilkS) (width 0.15))
+    (fp_line (start 0.5 0.5) (end -0.4 0) (layer B.SilkS) (width 0.15))
+    (fp_line (start -0.5 -0.5) (end -0.5 0.5) (layer B.SilkS) (width 0.15))
+    (fp_line (start -0.4 0) (end 0.5 -0.5) (layer F.SilkS) (width 0.15))
+    (fp_line (start 0.5 -0.5) (end 0.5 0.5) (layer F.SilkS) (width 0.15))
+    (fp_line (start 0.5 0.5) (end -0.4 0) (layer F.SilkS) (width 0.15))
+    (fp_line (start -0.5 -0.5) (end -0.5 0.5) (layer F.SilkS) (width 0.15))
+    (fp_line (start 2.7 -0.75) (end -2.7 -0.75) (layer F.SilkS) (width 0.15))
+    (fp_line (start -2.7 -0.75) (end -2.7 0.75) (layer F.SilkS) (width 0.15))
+    (fp_line (start -2.7 0.75) (end 2.7 0.75) (layer F.SilkS) (width 0.15))
+    (fp_line (start 2.7 0.75) (end 2.7 -0.75) (layer F.SilkS) (width 0.15))
+    (fp_line (start 2.7 -0.75) (end -2.7 -0.75) (layer B.SilkS) (width 0.15))
+    (fp_line (start -2.7 -0.75) (end -2.7 0.75) (layer B.SilkS) (width 0.15))
+    (fp_line (start -2.7 0.75) (end 2.7 0.75) (layer B.SilkS) (width 0.15))
+    (fp_line (start 2.7 0.75) (end 2.7 -0.75) (layer B.SilkS) (width 0.15))
+    (pad 1 smd rect (at -1.775 0 90) (size 1.3 0.95) (layers F.Cu F.Paste F.Mask)
+      (net 30 row3))
+    (pad 2 smd rect (at 1.775 0 90) (size 1.3 0.95) (layers B.Cu B.Paste B.Mask)
+      (net 57 "Net-(D34-Pad2)"))
+    (pad 1 smd rect (at -1.775 0 90) (size 1.3 0.95) (layers B.Cu B.Paste B.Mask)
+      (net 30 row3))
+    (pad 1 thru_hole rect (at -3.81 0 90) (size 1.397 1.397) (drill 0.8128) (layers *.Cu *.Mask F.SilkS)
+      (net 30 row3))
+    (pad 2 thru_hole circle (at 3.81 0 90) (size 1.397 1.397) (drill 0.8128) (layers *.Cu *.Mask F.SilkS)
+      (net 57 "Net-(D34-Pad2)"))
+    (pad 2 smd rect (at 1.775 0 90) (size 1.3 0.95) (layers F.Cu F.Paste F.Mask)
+      (net 57 "Net-(D34-Pad2)"))
+    (model Diodes_SMD.3dshapes/SMB_Handsoldering.wrl
+      (at (xyz 0 0 0))
+      (scale (xyz 0.22 0.15 0.15))
+      (rotate (xyz 0 0 180))
+    )
+  )
+  (module MX_Alps_Hybrid:MX-1U-NoLED (layer F.Cu)
+    (at 171.45 90.4875)
+    (fp_text reference SW35 (at 0 3.175) (layer F.SilkS)
+      (effects (font (size 1 1) (thickness 0.15)))
+    )
+    (fp_text value SW_PUSH (at 0 -7.9375) (layer Dwgs.User)
+      (effects (font (size 1 1) (thickness 0.15)))
+    )
+    (fp_line (start 5 -7) (end 7 -7) (layer Dwgs.User) (width 0.15))
+    (fp_line (start 7 -7) (end 7 -5) (layer Dwgs.User) (width 0.15))
+    (fp_line (start 5 7) (end 7 7) (layer Dwgs.User) (width 0.15))
+    (fp_line (start 7 7) (end 7 5) (layer Dwgs.User) (width 0.15))
+    (fp_line (start -7 5) (end -7 7) (layer Dwgs.User) (width 0.15))
+    (fp_line (start -7 7) (end -5 7) (layer Dwgs.User) (width 0.15))
+    (fp_line (start -5 -7) (end -7 -7) (layer Dwgs.User) (width 0.15))
+    (fp_line (start -7 -7) (end -7 -5) (layer Dwgs.User) (width 0.15))
+    (fp_line (start -9.525 -9.525) (end 9.525 -9.525) (layer Dwgs.User) (width 0.15))
+    (fp_line (start 9.525 -9.525) (end 9.525 9.525) (layer Dwgs.User) (width 0.15))
+    (fp_line (start 9.525 9.525) (end -9.525 9.525) (layer Dwgs.User) (width 0.15))
+    (fp_line (start -9.525 9.525) (end -9.525 -9.525) (layer Dwgs.User) (width 0.15))
+    (pad 2 thru_hole oval (at 2.5 -4.5 86.0548) (size 2.831378 2.25) (drill 1.47 (offset 0.290689 0)) (layers *.Cu B.Mask)
+      (net 57 "Net-(D34-Pad2)"))
+    (pad 2 thru_hole circle (at 2.54 -5.08) (size 2.25 2.25) (drill 1.47) (layers *.Cu B.Mask)
+      (net 57 "Net-(D34-Pad2)"))
+    (pad 1 thru_hole oval (at -3.81 -2.54 48.0996) (size 4.211556 2.25) (drill 1.47 (offset 0.980778 0)) (layers *.Cu B.Mask)
+      (net 50 col7))
+    (pad "" np_thru_hole circle (at 0 0) (size 3.9878 3.9878) (drill 3.9878) (layers *.Cu *.Mask))
+    (pad 1 thru_hole circle (at -2.5 -4) (size 2.25 2.25) (drill 1.47) (layers *.Cu B.Mask)
+      (net 50 col7))
+    (pad "" np_thru_hole circle (at -5.08 0 48.0996) (size 1.75 1.75) (drill 1.75) (layers *.Cu *.Mask))
+    (pad "" np_thru_hole circle (at 5.08 0 48.0996) (size 1.75 1.75) (drill 1.75) (layers *.Cu *.Mask))
+  )
   (gr_text "iroha60 rev.1\nDesigned by kironono" (at 98.575 116.0375) (layer F.SilkS)
     (effects (font (size 1.5 1.5) (thickness 0.3)))
@@
   (segment (start 134.3625 56.66) (end 134.825 56.1975) (width 0.25) (layer F.Cu) (net 11))
   (segment (start 134.3625 57.7625) (end 134.3625 56.66) (width 0.25) (layer F.Cu) (net 11))
+  (segment (start 131.825 56.1975) (end 134.825 56.1975) (width 0.25) (layer F.Cu) (net 11))
   (segment (start 50.815 48.5775) (end 55.625 48.5775) (width 0.25) (layer F.Cu) (net 12))
   (segment (start 50.125 47.8875) (end 50.815 48.5775) (width 0.25) (layer F.Cu) (net 12))
@@
   (segment (start 156.0625 48.3625) (end 156.0625 51.1625) (width 0.25) (layer B.Cu) (net 30))
   (via (at 155.1625 79.5625) (size 0.8) (drill 0.4) (layers F.Cu B.Cu) (net 30))
-  (segment (start 154.20475 94.2975) (end 153.25625 94.2975) (width 0.25) (layer F.Cu) (net 30))
   (segment (start 155.1625 93.33975) (end 154.20475 94.2975) (width 0.25) (layer F.Cu) (net 30))
   (segment (start 155.1625 79.5625) (end 155.1625 93.33975) (width 0.25) (layer F.Cu) (net 30))
@@
   (segment (start 155.8625 51.3625) (end 145.2625 61.9625) (width 0.25) (layer F.Cu) (net 30))
   (segment (start 145.2625 61.9625) (end 145.2625 74.687521) (width 0.25) (layer F.Cu) (net 30))
+  (segment (start 163.45 92.2625) (end 163.45 94.2975) (width 0.25) (layer F.Cu) (net 30))
+  (segment (start 163.45 92.2625) (end 163.45 94.2975) (width 0.25) (layer B.Cu) (net 30))
+  (segment (start 154.20475 94.2975) (end 163.45 94.2975) (width 0.25) (layer F.Cu) (net 30))
+  (segment (start 153.25625 94.2975) (end 154.20475 94.2975) (width 0.25) (layer F.Cu) (net 30))
   (segment (start 103.2025 86.6775) (end 108.0125 86.6775) (width 0.25) (layer F.Cu) (net 31))
   (segment (start 102.5125 85.9875) (end 103.2025 86.6775) (width 0.25) (layer F.Cu) (net 31))
@@
   (segment (start 159.164089 50.012511) (end 149.987499 59.189101) (width 0.25) (layer F.Cu) (net 50))
   (segment (start 162.712489 50.012511) (end 159.164089 50.012511) (width 0.25) (layer F.Cu) (net 50))
+  (via (at 162.35 74.2875) (size 0.8) (drill 0.4) (layers F.Cu B.Cu) (net 50))
+  (segment (start 162.35 70.811776) (end 162.35 74.2875) (width 0.25) (layer F.Cu) (net 50))
+  (segment (start 160.435724 68.8975) (end 162.35 70.811776) (width 0.25) (layer F.Cu) (net 50))
+  (segment (start 155.73375 68.8975) (end 160.435724 68.8975) (width 0.25) (layer F.Cu) (net 50))
+  (via (at 159.75 76.7875) (size 0.8) (drill 0.4) (layers F.Cu B.Cu) (net 50))
+  (segment (start 159.85 76.7875) (end 159.75 76.7875) (width 0.25) (layer B.Cu) (net 50))
+  (segment (start 162.35 74.2875) (end 159.85 76.7875) (width 0.25) (layer B.Cu) (net 50))
+  (segment (start 162.75 76.7875) (end 168.95 82.9875) (width 0.25) (layer F.Cu) (net 50))
+  (via (at 168.95 82.9875) (size 0.8) (drill 0.4) (layers F.Cu B.Cu) (net 50))
+  (segment (start 159.75 76.7875) (end 162.75 76.7875) (width 0.25) (layer F.Cu) (net 50))
+  (segment (start 168.95 82.9875) (end 168.95 86.4875) (width 0.25) (layer B.Cu) (net 50))
   (segment (start 177.218749 65.084349) (end 172.847499 60.713099) (width 0.25) (layer F.Cu) (net 51))
   (segment (start 177.218749 73.362499) (end 177.218749 65.084349) (width 0.25) (layer F.Cu) (net 51))
   (segment (start 172.847499 60.713099) (end 172.0855 59.9511) (width 0.25) (layer F.Cu) (net 51))
   (segment (start 178.54375 74.6875) (end 177.218749 73.362499) (width 0.25) (layer F.Cu) (net 51))
+  (segment (start 163.45 88.7125) (end 163.45 86.6775) (width 0.25) (layer F.Cu) (net 57))
+  (segment (start 163.45 88.7125) (end 163.45 86.6775) (width 0.25) (layer B.Cu) (net 57))
+  (segment (start 172.865001 84.282501) (end 173.99 85.4075) (width 0.25) (layer F.Cu) (net 57))
+  (segment (start 166.832827 84.282501) (end 172.865001 84.282501) (width 0.25) (layer F.Cu) (net 57))
+  (segment (start 164.437828 86.6775) (end 166.832827 84.282501) (width 0.25) (layer F.Cu) (net 57))
+  (segment (start 163.45 86.6775) (end 164.437828 86.6775) (width 0.25) (layer F.Cu) (net 57))
   (zone (net 0) (net_name "") (layer F.Cu) (hatch edge 0.508)
     (connect_pads (clearance 0.508))

Commit message: Updated
Parts:
- moved G*** 14.7 mm to (157.2, 110.3)
