File: iroha60/pcb/iroha60-right/iroha60-right.kicad_pcb (KiCad board)
At the start: 2 copper layers, 161.9 x 95.2 mm, 80 parts, among them J1 MJ-4PP-9, J2 LED, SW1 SW_PUSH, SW10 SW_PUSH, SW11 SW_PUSH, SW12 SW_PUSH, SW13 SW_PUSH, SW14 SW_PUSH, SW15 SW_PUSH, SW16 SW_PUSH, SW17 SW_PUSH, SW18 SW_PUSH, SW19 SW_PUSH, SW2 SW_PUSH, SW20 SW_PUSH, SW21 SW_PUSH, SW22 SW_PUSH, SW23 SW_PUSH, SW24 SW_PUSH, SW25 SW_PUSH, SW26 SW_PUSH, SW27 SW_PUSH, SW28 SW_PUSH, SW29 SW_PUSH, SW3 SW_PUSH, SW30 SW_PUSH, SW31 SW_PUSH, SW32 SW_PUSH, SW33 SW_PUSH, SW34 RESET_SW, SW35 SW_PUSH, SW4 SW_PUSH, SW5 SW_PUSH, SW6 SW_PUSH, SW7 SW_PUSH, SW8 SW_PUSH, SW9 SW_PUSH, U1 ProMicro

Commit message: Updated
Parts:
- SW23: footprint MX_Alps_Hybrid:MX-2.25U-ReversedStabilizers-NoLED -> MX_Alps_Hybrid:MX-2.25U-NoLED
- moved D23 28.0 mm to (139.5, 71.4)
- moved D31 12.0 mm to (84.3, 109.5)
Routing:
- net Net-(D23-Pad2): track 9.86 -> 31.0 mm, vias 0 -> 4
- net Net-(D31-Pad2): track 9.86 -> 21.9 mm
- net row2: track 192.8 -> 188.6 mm
- net row4: track 181.3 -> 185.2 mm
- net led: track 159.3 -> 161.7 mm
- net col5: track 114.7 -> 112.7 mm
- net col4: track 168.2 -> 169.8 mm
- net row3: track 203.3 -> 204.4 mm

Commit message: Updated
Other:
- board text added: "iroha60 rev.1 2020-08-12 Designed by kironono"
- board text removed: "iroha60 rev.1 Designed by kironono"
Changed lines of the file:
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@@
     (arrow2b (pts (xy 180.975 16.66875) (xy 179.848496 17.255171)))
   )
-  (gr_text "iroha60 rev.1\nDesigned by kironono" (at 98.575 116.0375) (layer F.SilkS)
+  (gr_text "iroha60 rev.1 2020-08-12\nDesigned by kironono" (at 98.575 116.0375) (layer F.SilkS)
     (effects (font (size 1.5 1.5) (thickness 0.3)))
   )
