File: iroha60/pcb/iroha60-right/iroha60-right.sch (KiCad schematic (older format))
At the start: 89 parts, among them J1 i2c-pin, J2 MJ-4PP-9, J3 i2c-pin, J4 LED, SW1 SW_PUSH, SW10 SW_PUSH, SW11 SW_PUSH, SW12 SW_PUSH, SW13 SW_PUSH, SW14 SW_PUSH, SW15 SW_PUSH, SW16 SW_PUSH, SW17 SW_PUSH, SW18 SW_PUSH, SW19 SW_PUSH, SW2 SW_PUSH, SW20 SW_PUSH, SW21 SW_PUSH, SW22 SW_PUSH, SW23 SW_PUSH, SW24 SW_PUSH, SW25 SW_PUSH, SW26 SW_PUSH, SW27 SW_PUSH, SW28 SW_PUSH, SW29 SW_PUSH, SW3 SW_PUSH, SW30 SW_PUSH, SW31 SW_PUSH, SW32 SW_PUSH, SW33 SW_PUSH, SW34 SW_PUSH, SW35 SW_PUSH, SW36 SW_PUSH, SW37 SW_PUSH, SW38 SW_PUSH, SW39 SW_PUSH, SW4 SW_PUSH, SW40 SW_PUSH, SW41 SW_PUSH, SW42 RESET_SW, SW5 SW_PUSH, SW6 SW_PUSH, SW7 SW_PUSH, SW8 SW_PUSH, SW9 SW_PUSH, U1 ProMicro

Commit message: Updated
Parts:
- D1, D10, D11, D12, D13, D14, D15, D16, D17, D18, D19, D2, D20, D21, D22, D23, D24, D25, D26, D27, D28, D29, D3, D30, D31, D32, D33, D34, D35, D36, D37, D38, D39, D4, D40, D41, D5, D6, D7, D8, D9: footprint (none) -> kbd:D3_TH_SMD
- J1, J3: footprint (none) -> kbd:1pin_conn
- J2: footprint (none) -> kbd:MJ-4PP-9_1side
- J4: footprint (none) -> kbd:StripLED_1side
- JP1: footprint (none) -> kbd:Jumper
- SW1, SW10, SW11, SW12, SW13, SW14, SW15, SW16, SW18, SW19, SW2, SW20, SW21, SW22, SW23, SW24, SW26, SW27, SW28, SW29, SW3, SW30, SW31, SW33, SW34, SW35, SW38, SW39, SW4, SW40, SW41, SW5, SW6, SW7, SW8, SW9: footprint (none) -> MX_Alps_Hybrid:MX-1U-NoLED
- SW17, SW37: footprint (none) -> MX_Alps_Hybrid:MX-1.5U-NoLED
- SW25, SW36: footprint (none) -> MX_Alps_Hybrid:MX-2.25U-ReversedStabilizers-NoLED
- SW32: footprint (none) -> MX_Alps_Hybrid:MX-1.75U-NoLED
- SW42: footprint (none) -> kbd:ResetSW_1side
- U1: footprint (none) -> kbd:ProMicro_v3.5

Commit message: Updated
Parts:
- removed D18, D26, D33, D34, D39, D40, D41, D9: D, kbd:D3_TH_SMD, symbol Device:D
- removed SW18, SW26, SW33, SW34, SW39, SW40, SW41, SW9: SW_PUSH, MX_Alps_Hybrid:MX-1U-NoLED, symbol kbd:SW_PUSH
- U1: footprint kbd:ProMicro_v3.5 -> kbd:ProMicro_v3
- renumbered D11 to D10, D12 to D11, D13 to D12, D14 to D13, D15 to D14, D16 to D15, D17 to D16, D19 to D17, D20 to D18, D21 to D19, D22 to D20, D23 to D21, D24 to D22, D25 to D23, D27 to D24, D28 to D25, D29 to D26, D30 to D27, D31 to D28, D32 to D29, D35 to D30, D36 to D31, D37 to D32, D38 to D33, D10 to D9, SW11 to SW10, SW12 to SW11, SW13 to SW12, SW14 to SW13, SW15 to SW14, SW16 to SW15, SW17 to SW16, SW19 to SW17, SW20 to SW18, SW21 to SW19, SW22 to SW20, SW23 to SW21, SW24 to SW22, SW25 to SW23, SW27 to SW24, SW28 to SW25, SW29 to SW26, SW30 to SW27, SW31 to SW28, SW32 to SW29, SW35 to SW30, SW36 to SW31, SW37 to SW32, SW38 to SW33, SW42 to SW34, SW10 to SW9
Connections:
- net col8: no longer names the net of U1.12 (9/B5)
- no-connect marks 3 -> 4
Other:
- moved on the sheet: U1

Commit message: Updated
Parts:
- removed J1, J3: i2c-pin, kbd:1pin_conn, symbol Connector_Generic:Conn_01x01
- removed JP1: Jumper, kbd:Jumper, symbol Device:Jumper
- U1: footprint kbd:ProMicro_v3 -> kbd:ProMicro_v2_1side
- renumbered J2 to J1, J4 to J2
Connections:
- net data: now also J1.B
- no-connect marks 4 -> 5
Changed lines of the file:
@@
 F 0 "U1" H 2025 7187 60  0000 C CNN
 F 1 "ProMicro" H 2025 7081 60  0000 C CNN
-F 2 "kbd:ProMicro_v3" H 2125 5100 60  0001 C CNN
+F 2 "kbd:ProMicro_v2_1side" H 2125 5100 60  0001 C CNN
 F 3 "" H 2125 5100 60  0000 C CNN
 	1    2025 6150
@@
 NoConn ~ 2725 5400
 $Comp
-L kbd:MJ-4PP-9 J2
+L kbd:MJ-4PP-9 J1
 U 1 1 5E052F2D
 P 5875 5475
-F 0 "J2" H 5906 5751 50  0000 C CNN
+F 0 "J1" H 5906 5751 50  0000 C CNN
 F 1 "MJ-4PP-9" H 5906 5660 50  0000 C CNN
 F 2 "kbd:MJ-4PP-9_1side" H 6150 5650 50  0001 C CNN
@@
 	1    5875 5475
 	1    0    0    -1
-$EndComp
-$Comp
-L Device:Jumper JP1
-U 1 1 5E053848
-P 7250 5550
-F 0 "JP1" H 7250 5325 50  0000 C CNN
-F 1 "Jumper" H 7250 5416 50  0000 C CNN
-F 2 "kbd:Jumper" H 7250 5550 50  0001 C CNN
-F 3 "~" H 7250 5550 50  0001 C CNN
-	1    7250 5550
-	-1   0    0    1
 $EndComp
 $Comp
@@
 $EndComp
 $Comp
-L Connector_Generic:Conn_01x01 J1
-U 1 1 5E056F6B
-P 6775 5125
-F 0 "J1" V 6739 5037 50  0000 R CNN
-F 1 "i2c-pin" V 6648 5037 50  0000 R CNN
-F 2 "kbd:1pin_conn" H 6775 5125 50  0001 C CNN
-F 3 "~" H 6775 5125 50  0001 C CNN
-	1    6775 5125
-	0    -1   -1   0
-$EndComp
-$Comp
-L Connector_Generic:Conn_01x01 J3
-U 1 1 5E057B6E
-P 6775 5925
-F 0 "J3" V 6647 6005 50  0000 L CNN
-F 1 "i2c-pin" V 6738 6005 50  0000 L CNN
-F 2 "kbd:1pin_conn" H 6775 5925 50  0001 C CNN
-F 3 "~" H 6775 5925 50  0001 C CNN
-	1    6775 5925
-	0    1    1    0
-$EndComp
-$Comp
-L Connector_Generic:Conn_01x03 J4
+L Connector_Generic:Conn_01x03 J2
 U 1 1 5E05841F
 P 4150 6450
-F 0 "J4" H 4068 6125 50  0000 C CNN
+F 0 "J2" H 4068 6125 50  0000 C CNN
 F 1 "LED" H 4068 6216 50  0000 C CNN
 F 2 "kbd:StripLED_1side" H 4150 6450 50  0001 C CNN
@@
 Wire Wire Line
 	6400 5500 6075 5500
-Wire Wire Line
-	6075 5400 6775 5400
-Wire Wire Line
-	6775 5400 6775 5325
-Wire Wire Line
-	6075 5550 6775 5550
-Wire Wire Line
-	6775 5550 6775 5725
-Wire Wire Line
-	6950 5550 6775 5550
-Connection ~ 6775 5550
-Text GLabel 7550 5550 2    50   Input ~ 0
+Text GLabel 6950 5550 2    50   Input ~ 0
 data
 Text GLabel 4350 6450 2    50   Input ~ 0
@@
 col7
 NoConn ~ 1325 6500
+Wire Wire Line
+	6075 5550 6950 5550
+NoConn ~ 6075 5400
 $EndSCHEMATC

Commit message: Updated
Parts:
- added D34: D, kbd:D3_TH_SMD, symbol Device:D
- added SW35: SW_PUSH, MX_Alps_Hybrid:MX-1U-NoLED, symbol kbd:SW_PUSH
Connections:
- net col7: now also SW35.1
- net row3: now also D34.1 (K)
- new net: D34.2 (A), SW35.2
Changed lines of the file:
@@
 	6075 5550 6950 5550
 NoConn ~ 6075 5400
+$Comp
+L kbd:SW_PUSH SW35
+U 1 1 5F1C08B5
+P 9325 3500
+F 0 "SW35" H 9325 3755 50  0000 C CNN
+F 1 "SW_PUSH" H 9325 3664 50  0000 C CNN
+F 2 "MX_Alps_Hybrid:MX-1U-NoLED" H 9325 3500 50  0001 C CNN
+F 3 "" H 9325 3500 50  0000 C CNN
+	1    9325 3500
+	1    0    0    -1
+$EndComp
+$Comp
+L Device:D D34
+U 1 1 5F1C08BF
+P 9625 3650
+F 0 "D34" V 9671 3571 50  0000 R CNN
+F 1 "D" V 9580 3571 50  0000 R CNN
+F 2 "kbd:D3_TH_SMD" H 9625 3650 50  0001 C CNN
+F 3 "~" H 9625 3650 50  0001 C CNN
+	1    9625 3650
+	0    -1   -1   0
+$EndComp
+Wire Wire Line
+	9625 3800 8775 3800
+Wire Wire Line
+	9025 3500 9025 2775
+Connection ~ 8775 3800
+Connection ~ 9025 2775
 $EndSCHEMATC

Commit message: Updated
Parts:
- SW23: footprint MX_Alps_Hybrid:MX-2.25U-ReversedStabilizers-NoLED -> MX_Alps_Hybrid:MX-2.25U-NoLED
Changed lines of the file:
@@
 F 0 "SW23" H 9325 3030 50  0000 C CNN
 F 1 "SW_PUSH" H 9325 2939 50  0000 C CNN
-F 2 "MX_Alps_Hybrid:MX-2.25U-ReversedStabilizers-NoLED" H 9325 2775 50  0001 C CNN
+F 2 "MX_Alps_Hybrid:MX-2.25U-NoLED" H 9325 2775 50  0001 C CNN
 F 3 "" H 9325 2775 50  0000 C CNN
 	1    9325 2775
